Commit message: Fix the macros and launch to include initial positions

File: yaskawa_ros2_control_support/urdf/common_macro.ros2_control.xacro (robot description, xacro)
@@ -8,5 +8,6 @@
                sim_gazebo:=^|false
                simulation_controllers
-               description_package"
+               description_package
+               initial_positions:=${dict(joint_1_s=0.0,joint_2_l=0.0,joint_3_u=1.57,joint_4_r=0.0,joint_5_b=1.57,joint_6_t=0.0)}"
                >
     <ros2_control name="${name}" type="system">
@@ -28,5 +29,5 @@
         </command_interface>
         <state_interface name="position">
-          <param name="initial_value">0</param>
+          <param name="initial_value">${initial_positions['joint_1_s']}</param>
         </state_interface>
       </joint>
@@ -37,5 +38,5 @@
         </command_interface>
         <state_interface name="position">
-          <param name="initial_value">0</param>
+          <param name="initial_value">${initial_positions['joint_2_l']}</param>
         </state_interface>
 	  </joint>
@@ -46,5 +47,5 @@
         </command_interface>
         <state_interface name="position">
-          <param name="initial_value">0</param>
+          <param name="initial_value">${initial_positions['joint_3_u']}</param>
         </state_interface>
 	  </joint>
@@ -55,5 +56,5 @@
         </command_interface>
         <state_interface name="position">
-          <param name="initial_value">0</param>
+          <param name="initial_value">${initial_positions['joint_4_r']}</param>
         </state_interface>
       </joint>
@@ -64,5 +65,5 @@
         </command_interface>
         <state_interface name="position">
-          <param name="initial_value">0</param>
+          <param name="initial_value">${initial_positions['joint_5_b']}</param>
         </state_interface>
       </joint>
@@ -73,5 +74,5 @@
         </command_interface>
         <state_interface name="position">
-          <param name="initial_value">0</param>
+          <param name="initial_value">${initial_positions['joint_6_t']}</param>
         </state_interface>
       </joint>

File: yaskawa_ros2_control_support/urdf/common_yaskawa.xacro (robot description, xacro)
@@ -10,8 +10,10 @@
   <xacro:arg name="sim_gazebo" default="false" />
   <xacro:arg name="simulation_controllers" default="" />
+  <xacro:arg name="initial_positions_file" default="$(find yaskawa_ros2_control_support)/config/initial_positions.yaml"/>
   <xacro:property name="description_package" value="$(arg description_package)"/>
   <xacro:property name="description_macro_file" value="$(arg description_macro_file)"/>
   <xacro:property name="robot_name" value="$(arg robot_name)"/>
   <!-- convert to property to use substitution in function -->
+  <xacro:property name="initial_positions_file" default="$(arg initial_positions_file)"/>
   <xacro:include filename="$(find ${description_package})/urdf/${description_macro_file}"/>
   <xacro:include filename="$(find yaskawa_ros2_control_support)/urdf/common_macro.ros2_control.xacro"/>
@@ -24,4 +26,5 @@
     simulation_controllers="$(arg simulation_controllers)"
     description_package="$(arg description_package)"
+    initial_positions="${xacro.load_yaml(initial_positions_file)}"
   />
   <xacro:if value="${description_package == 'motoman_gp250_support'}">
