Commit message: added visual and collision meshes for gp280

File: motoman_gp280_support/urdf/gp280_macro.xacro (robot description, xacro)
@@ -7,5 +7,5 @@
         <visual>
             <geometry>
-                <mesh filename="package://motoman_gp280_support/meshes/gp280/visual/base_link.stl"/>
+                <mesh filename="package://motoman_gp280_support/meshes/gp280/visual/base_link_visual.stl"/>
             </geometry>
             <xacro:material_yaskawa_blue/>
@@ -13,5 +13,5 @@
         <collision>
             <geometry>
-                <mesh filename="package://motoman_gp280_support/meshes/gp280/collision/base_link.stl"/>
+                <mesh filename="package://motoman_gp280_support/meshes/gp280/collision/base_link_collision.stl"/>
             </geometry>
         </collision>
@@ -20,5 +20,5 @@
         <visual>
             <geometry>
-                <mesh filename="package://motoman_gp280_support/meshes/gp280/visual/link_1_s.stl"/>
+                <mesh filename="package://motoman_gp280_support/meshes/gp280/visual/link_1_s_visual.stl"/>
             </geometry>
             <xacro:material_yaskawa_blue/>
@@ -26,5 +26,5 @@
         <collision>
             <geometry>
-                <mesh filename="package://motoman_gp280_support/meshes/gp280/collision/link_1_s.stl"/>
+                <mesh filename="package://motoman_gp280_support/meshes/gp280/collision/link_1_s_collision.stl"/>
             </geometry>
         </collision>
@@ -33,5 +33,5 @@
         <visual>
             <geometry>
-                <mesh filename="package://motoman_gp280_support/meshes/gp280/visual/link_2_l.stl"/>
+                <mesh filename="package://motoman_gp280_support/meshes/gp280/visual/link_2_l_visual.stl"/>
             </geometry>
             <xacro:material_yaskawa_blue/>
@@ -39,5 +39,5 @@
         <collision>
             <geometry>
-                <mesh filename="package://motoman_gp280_support/meshes/gp280/collision/link_2_l.stl"/>
+                <mesh filename="package://motoman_gp280_support/meshes/gp280/collision/link_2_l_no_balancer_collision.stl"/>
             </geometry>
         </collision>
@@ -46,5 +46,5 @@
         <visual>
             <geometry>
-                <mesh filename="package://motoman_gp280_support/meshes/gp280/visual/link_3_u.stl"/>
+                <mesh filename="package://motoman_gp280_support/meshes/gp280/visual/link_3_u_visual.stl"/>
             </geometry>
             <xacro:material_yaskawa_blue/>
@@ -52,5 +52,5 @@
         <collision>
             <geometry>
-                <mesh filename="package://motoman_gp280_support/meshes/gp280/collision/link_3_u.stl"/>
+                <mesh filename="package://motoman_gp280_support/meshes/gp280/collision/link_3_u_collision.stl"/>
             </geometry>
         </collision>
@@ -59,5 +59,5 @@
         <visual>
             <geometry>
-                <mesh filename="package://motoman_gp280_support/meshes/gp280/visual/link_4_r.stl"/>
+                <mesh filename="package://motoman_gp280_support/meshes/gp280/visual/link_4_r_visual.stl"/>
             </geometry>
             <xacro:material_yaskawa_blue/>
@@ -65,5 +65,5 @@
         <collision>
             <geometry>
-                <mesh filename="package://motoman_gp280_support/meshes/gp280/collision/link_4_r.stl"/>
+                <mesh filename="package://motoman_gp280_support/meshes/gp280/collision/link_4_r_collision.stl"/>
             </geometry>
         </collision>
@@ -72,5 +72,5 @@
         <visual>
             <geometry>
-                <mesh filename="package://motoman_gp280_support/meshes/gp280/visual/link_5_b.stl"/>
+                <mesh filename="package://motoman_gp280_support/meshes/gp280/visual/link_5_b_visual.stl"/>
             </geometry>
             <xacro:material_yaskawa_blue/>
@@ -78,5 +78,5 @@
         <collision>
             <geometry>
-                <mesh filename="package://motoman_gp280_support/meshes/gp280/collision/link_5_b.stl"/>
+                <mesh filename="package://motoman_gp280_support/meshes/gp280/collision/link_5_b_collision.stl"/>
             </geometry>
         </collision>
@@ -85,5 +85,5 @@
         <visual>
             <geometry>
-                <mesh filename="package://motoman_gp280_support/meshes/gp280/visual/link_6_t.stl"/>
+                <mesh filename="package://motoman_gp280_support/meshes/gp280/visual/link_6_t_visual.stl"/>
             </geometry>
             <xacro:material_yaskawa_blue/>
@@ -91,5 +91,5 @@
         <collision>
             <geometry>
-                <mesh filename="package://motoman_gp280_support/meshes/gp280/collision/link_6_t.stl"/>
+                <mesh filename="package://motoman_gp280_support/meshes/gp280/collision/link_6_t_collision.stl"/>
             </geometry>
         </collision>
