Commit message: Updated files to work with proper joint names.

File: motoman_common_moveit/srdf/common_motoman.srdf.xacro (robot description, xacro)
@@ -5,5 +5,5 @@
 -->
 <robot name="$(arg robot_name)" xmlns:xacro="http://wiki.ros.org/xacro">
-    <xacro:arg name="robot_name" default="yaskawa"/>
+    <xacro:arg name="robot_name" default="motoman"/>
     <xacro:arg name="prefix" default="" />
     <!--GROUPS- Representation of a set of joints and links. This can be useful for specifying DOF to plan for, defining arms, end effectors, etc-->
@@ -13,10 +13,10 @@
     <!--SUBGROUPS- Groups can also be formed by referencing to already defined group names-->
     <group name="manipulator">
-        <chain base_link="base_link" tip_link="$(arg prefix)tool0"/>
+        <chain base_link="$(arg prefix)base_link" tip_link="$(arg prefix)tool0"/>
     </group>
     <group_state name="home" group="manipulator">
         <joint name="$(arg prefix)joint_1" value="0"/>
-        <joint name="$(arg prefix)joint_2" value="-1.57"/>
-        <joint name="$(arg prefix)joint_3" value="1.57"/>
+        <joint name="$(arg prefix)joint_2" value="0"/>
+        <joint name="$(arg prefix)joint_3" value="0"/>
         <joint name="$(arg prefix)joint_4" value="0"/>
         <joint name="$(arg prefix)joint_5" value="1.57"/>
@@ -24,17 +24,17 @@
     </group_state>
     <!--DISABLE COLLISIONS- By default it is assumed that any link of the robot could potentially come into collision with any other link in the robot. This tag disables collision checking between a specified pair of links. -->
-    <disable_collisions link1="base_link" link2="$(arg prefix)link_1_s" reason="Adjacent"/>
-    <disable_collisions link1="base_link" link2="$(arg prefix)link_2_l" reason="Never"/>
-    <disable_collisions link1="base_link" link2="$(arg prefix)link_3_u" reason="Never"/>
-    <disable_collisions link1="$(arg prefix)link_1_s" link2="$(arg prefix)link_2_l" reason="Adjacent"/>
-    <disable_collisions link1="$(arg prefix)link_1_s" link2="$(arg prefix)link_3_u" reason="Never"/>
-    <disable_collisions link1="$(arg prefix)link_2_l" link2="$(arg prefix)link_3_u" reason="Adjacent"/>
-    <disable_collisions link1="$(arg prefix)link_2_l" link2="$(arg prefix)link_4_r" reason="Never"/>
-    <disable_collisions link1="$(arg prefix)link_2_l" link2="$(arg prefix)link_5_b" reason="Never"/>
-    <disable_collisions link1="$(arg prefix)link_2_l" link2="$(arg prefix)link_6_t" reason="Never"/>
-    <disable_collisions link1="$(arg prefix)link_3_u" link2="$(arg prefix)link_4_r" reason="Adjacent"/>
-    <disable_collisions link1="$(arg prefix)link_3_u" link2="$(arg prefix)link_5_b" reason="Never"/>
-    <disable_collisions link1="$(arg prefix)link_3_u" link2="$(arg prefix)link_6_t" reason="Never"/>
-    <disable_collisions link1="$(arg prefix)link_4_r" link2="$(arg prefix)link_5_b" reason="Adjacent"/>
-    <disable_collisions link1="$(arg prefix)link_5_b" link2="$(arg prefix)link_6_t" reason="Adjacent"/>
+    <disable_collisions link1="$(arg prefix)base_link" link2="$(arg prefix)link_1" reason="Adjacent"/>
+    <disable_collisions link1="$(arg prefix)base_link" link2="$(arg prefix)link_2" reason="Never"/>
+    <disable_collisions link1="$(arg prefix)base_link" link2="$(arg prefix)link_3" reason="Never"/>
+    <disable_collisions link1="$(arg prefix)link_1" link2="$(arg prefix)link_2" reason="Adjacent"/>
+    <disable_collisions link1="$(arg prefix)link_1" link2="$(arg prefix)link_3" reason="Never"/>
+    <disable_collisions link1="$(arg prefix)link_2" link2="$(arg prefix)link_3" reason="Adjacent"/>
+    <disable_collisions link1="$(arg prefix)link_2" link2="$(arg prefix)link_4" reason="Never"/>
+    <disable_collisions link1="$(arg prefix)link_2" link2="$(arg prefix)link_5" reason="Never"/>
+    <disable_collisions link1="$(arg prefix)link_2" link2="$(arg prefix)link_6" reason="Never"/>
+    <disable_collisions link1="$(arg prefix)link_3" link2="$(arg prefix)link_4" reason="Adjacent"/>
+    <disable_collisions link1="$(arg prefix)link_3" link2="$(arg prefix)link_5" reason="Never"/>
+    <disable_collisions link1="$(arg prefix)link_3" link2="$(arg prefix)link_6" reason="Never"/>
+    <disable_collisions link1="$(arg prefix)link_4" link2="$(arg prefix)link_5" reason="Adjacent"/>
+    <disable_collisions link1="$(arg prefix)link_5" link2="$(arg prefix)link_6" reason="Adjacent"/>
 </robot>

File: motoman_gp250_support/urdf/gp250.xacro (robot description, xacro)
@@ -1,5 +1,13 @@
 <?xml version="1.0" ?>
-<robot name="motoman_gp250" xmlns:xacro="http://ros.org/wiki/xacro">
+<robot name="$(arg robot_name)" xmlns:xacro="http://ros.org/wiki/xacro">
+  <xacro:arg name="robot_name" default="motoman" />
+  <xacro:arg name="prefix" default="" />
+  <link name="world" />
+  <joint name="$(arg prefix)base_link-world" type="fixed">
+    <origin xyz="0 0 0" rpy="0 0 0"/>
+    <parent link="$(arg prefix)base_link"/>
+    <child link="world"/>
+  </joint>
   <xacro:include filename="$(find motoman_gp250_support)/urdf/gp250_macro.xacro" />
-  <xacro:motoman_gp250 prefix=""/>
+  <xacro:motoman_gp250 prefix="$(arg prefix)"/>
 </robot>

File: motoman_gp250_support/urdf/gp250_macro.xacro (robot description, xacro)
@@ -4,5 +4,5 @@
     <xacro:include filename="$(find motoman_resources)/urdf/common_materials.xacro"/>
     <!-- link list -->
-    <link name="base_link">
+    <link name="${prefix}base_link">
         <visual>
             <geometry>
@@ -17,5 +17,5 @@
         </collision>
     </link>
-    <link name="${prefix}link_1_s">
+    <link name="${prefix}link_1">
         <visual>
             <geometry>
@@ -30,5 +30,5 @@
         </collision>
     </link>
-    <link name="${prefix}link_2_l">
+    <link name="${prefix}link_2">
         <visual>
             <geometry>
@@ -43,5 +43,5 @@
         </collision>
     </link>
-    <link name="${prefix}link_3_u">
+    <link name="${prefix}link_3">
         <visual>
             <geometry>
@@ -56,5 +56,5 @@
         </collision>
     </link>
-    <link name="${prefix}link_4_r">
+    <link name="${prefix}link_4">
         <visual>
             <geometry>
@@ -69,5 +69,5 @@
         </collision>
     </link>
-    <link name="${prefix}link_5_b">
+    <link name="${prefix}link_5">
         <visual>
             <geometry>
@@ -82,5 +82,5 @@
         </collision>
     </link>
-    <link name="${prefix}link_6_t">
+    <link name="${prefix}link_6">
         <visual>
             <geometry>
@@ -99,6 +99,6 @@
     <!-- joint list -->
     <joint name="${prefix}joint_1" type="revolute">
-        <parent link="base_link"/>
-        <child link="${prefix}link_1_s"/>
+        <parent link="${prefix}base_link"/>
+        <child link="${prefix}link_1"/>
         <origin xyz="0 0 0.650" rpy="0 0 0" />
         <axis xyz="0 0 1" />
@@ -106,6 +106,6 @@
     </joint>
     <joint name="${prefix}joint_2" type="revolute">
-        <parent link="${prefix}link_1_s"/>
-        <child link="${prefix}link_2_l"/>
+        <parent link="${prefix}link_1"/>
+        <child link="${prefix}link_2"/>
         <origin xyz="0.285 0 0" rpy="0 0 0" />
         <axis xyz="0 1 0" />
@@ -113,6 +113,6 @@
     </joint>
     <joint name="${prefix}joint_3" type="revolute">
-        <parent link="${prefix}link_2_l"/>
-        <child link="${prefix}link_3_u"/>
+        <parent link="${prefix}link_2"/>
+        <child link="${prefix}link_3"/>
         <origin xyz="0 0 1.150" rpy="0 0 0" />
         <axis xyz="0 -1 0" />
@@ -120,6 +120,6 @@
     </joint>
     <joint name="${prefix}joint_4" type="revolute">
-        <parent link="${prefix}link_3_u"/>
-        <child link="${prefix}link_4_r"/>
+        <parent link="${prefix}link_3"/>
+        <child link="${prefix}link_4"/>
         <origin xyz="0 0 0.250" rpy="0 0 0" />
         <axis xyz="-1 0 0" />
@@ -127,6 +127,6 @@
     </joint>
     <joint name="${prefix}joint_5" type="revolute">
-        <parent link="${prefix}link_4_r"/>
-        <child link="${prefix}link_5_b"/>
+        <parent link="${prefix}link_4"/>
+        <child link="${prefix}link_5"/>
         <origin xyz="1.285 0 0" rpy="0 0 0" />
         <axis xyz="0 -1 0" />
@@ -134,6 +134,6 @@
     </joint>
     <joint name="${prefix}joint_6" type="revolute">
-        <parent link="${prefix}link_5_b"/>
-        <child link="${prefix}link_6_t"/>
+        <parent link="${prefix}link_5"/>
+        <child link="${prefix}link_6"/>
         <origin xyz="0 0 0" rpy="0 0 0" />
         <axis xyz="-1 0 0" />
@@ -142,5 +142,5 @@
     <joint name="${prefix}joint_6-tool0" type="fixed">
         <origin xyz="0.250 0 0" rpy="3.1415926 -1.570796 0"/>
-        <parent link="${prefix}link_6_t"/>
+        <parent link="${prefix}link_6"/>
         <child link="${prefix}tool0"/>
     </joint>
@@ -149,5 +149,5 @@
     <joint name="${prefix}joint_6-flange" type="fixed">
         <origin xyz="0 0 0" rpy="0 ${radians(90)} 0" />
-        <parent link="${prefix}link_6_t" />
+        <parent link="${prefix}link_6" />
         <child link="${prefix}flange" />
     </joint>
@@ -156,5 +156,5 @@
     <joint name="${prefix}base_link-base" type="fixed">
         <origin xyz="0 0 0.650" rpy="0 0 0"/>
-        <parent link="base_link"/>
+        <parent link="${prefix}base_link"/>
         <child link="${prefix}base"/>
     </joint>

File: motoman_ros2_control_support/urdf/common_macro.ros2_control.xacro (robot description, xacro)
@@ -24,6 +24,4 @@
     <joint name="${prefix}joint_1">
         <command_interface name="position">
-          <param name="min">-1</param>
-          <param name="max">1</param>
         </command_interface>
         <state_interface name="position">
@@ -33,6 +31,4 @@
       <joint name="${prefix}joint_2">
         <command_interface name="position">
-          <param name="min">-1</param>
-          <param name="max">1</param>
         </command_interface>
         <state_interface name="position">
@@ -42,6 +38,4 @@
       <joint name="${prefix}joint_3">
         <command_interface name="position">
-          <param name="min">-1</param>
-          <param name="max">0.61</param>
         </command_interface>
         <state_interface name="position">
@@ -51,6 +45,4 @@
       <joint name="${prefix}joint_4">
         <command_interface name="position">
-          <param name="min">-1</param>
-          <param name="max">1</param>
         </command_interface>
         <state_interface name="position">
@@ -60,6 +52,4 @@
       <joint name="${prefix}joint_5">
         <command_interface name="position">
-          <param name="min">-1</param>
-          <param name="max">1</param>
         </command_interface>
         <state_interface name="position">
@@ -69,6 +59,4 @@
       <joint name="${prefix}joint_6">
         <command_interface name="position">
-          <param name="min">-1</param>
-          <param name="max">1</param>
         </command_interface>
         <state_interface name="position">
