Commit message: Add mh5 support and modify common_moveit

File: motoman_common_moveit/srdf/common_yaskawa.srdf.xacro (robot description, xacro)
@@ -17,8 +17,8 @@
     <group_state name="home" group="manipulator">
         <joint name="$(arg prefix)joint_1" value="0"/>
-        <joint name="$(arg prefix)joint_2" value="-1.57"/>
-        <joint name="$(arg prefix)joint_3" value="1.57"/>
+        <joint name="$(arg prefix)joint_2" value="0"/>
+        <joint name="$(arg prefix)joint_3" value="0"/>
         <joint name="$(arg prefix)joint_4" value="0"/>
-        <joint name="$(arg prefix)joint_5" value="1.57"/>
+        <joint name="$(arg prefix)joint_5" value="0"/>
         <joint name="$(arg prefix)joint_6" value="0"/>
     </group_state>

File: motoman_mh5_support/urdf/mh5_macro.xacro (robot description, xacro)
@@ -133,9 +133,4 @@
 			<origin xyz="0 0 0.3100" rpy="0 0 0"/>
 			<axis xyz="0 -1 0" />
-      <!-- Old limits: lower="-2.3736" upper="4.4506" The new limits
-           below were measured from an MH5F.  They ensure that link_r
-           won't hit link_l even when joint_r is at 45 degrees.  The
-           old limits were converted directly from the MH5 data sheet,
-           which was clearly way off. -->
 			<limit lower="-1.0122" upper="3.2218" effort="100" velocity="2.96" />
 		</joint>
