Commit message: Add gp250 support and set it as default

File: motoman_gp250_support/urdf/gp250_macro.xacro (robot description, xacro)
@@ -1,5 +1,5 @@
 <?xml version="1.0" ?>
 <robot xmlns:xacro="http://ros.org/wiki/xacro">
-  <xacro:macro name="motoman_gp280" params="prefix">
+  <xacro:macro name="motoman_gp250" params="prefix">
     <xacro:include filename="$(find motoman_resources)/urdf/common_materials.xacro"/>
     <!-- link list -->
@@ -7,5 +7,5 @@
         <visual>
             <geometry>
-                <mesh filename="package://motoman_gp280_support/meshes/gp280/visual/base_link.stl"/>
+                <mesh filename="package://motoman_gp250_support/meshes/gp250/visual/base_link.stl"/>
             </geometry>
             <xacro:material_yaskawa_blue/>
@@ -13,5 +13,5 @@
         <collision>
             <geometry>
-                <mesh filename="package://motoman_gp280_support/meshes/gp280/collision/base_link.stl"/>
+                <mesh filename="package://motoman_gp250_support/meshes/gp250/collision/base_link.stl"/>
             </geometry>
         </collision>
@@ -20,5 +20,5 @@
         <visual>
             <geometry>
-                <mesh filename="package://motoman_gp280_support/meshes/gp280/visual/link_1_s.stl"/>
+                <mesh filename="package://motoman_gp250_support/meshes/gp250/visual/link_1_s.stl"/>
             </geometry>
             <xacro:material_yaskawa_blue/>
@@ -26,5 +26,5 @@
         <collision>
             <geometry>
-                <mesh filename="package://motoman_gp280_support/meshes/gp280/collision/link_1_s.stl"/>
+                <mesh filename="package://motoman_gp250_support/meshes/gp250/collision/link_1_s.stl"/>
             </geometry>
         </collision>
@@ -33,5 +33,5 @@
         <visual>
             <geometry>
-                <mesh filename="package://motoman_gp280_support/meshes/gp280/visual/link_2_l.stl"/>
+                <mesh filename="package://motoman_gp250_support/meshes/gp250/visual/link_2_l.stl"/>
             </geometry>
             <xacro:material_yaskawa_blue/>
@@ -39,5 +39,5 @@
         <collision>
             <geometry>
-                <mesh filename="package://motoman_gp280_support/meshes/gp280/collision/link_2_l.stl"/>
+                <mesh filename="package://motoman_gp250_support/meshes/gp250/collision/link_2_l.stl"/>
             </geometry>
         </collision>
@@ -46,5 +46,5 @@
         <visual>
             <geometry>
-                <mesh filename="package://motoman_gp280_support/meshes/gp280/visual/link_3_u.stl"/>
+                <mesh filename="package://motoman_gp250_support/meshes/gp250/visual/link_3_u.stl"/>
             </geometry>
             <xacro:material_yaskawa_blue/>
@@ -52,5 +52,5 @@
         <collision>
             <geometry>
-                <mesh filename="package://motoman_gp280_support/meshes/gp280/collision/link_3_u.stl"/>
+                <mesh filename="package://motoman_gp250_support/meshes/gp250/collision/link_3_u.stl"/>
             </geometry>
         </collision>
@@ -59,5 +59,5 @@
         <visual>
             <geometry>
-                <mesh filename="package://motoman_gp280_support/meshes/gp280/visual/link_4_r.stl"/>
+                <mesh filename="package://motoman_gp250_support/meshes/gp250/visual/link_4_r.stl"/>
             </geometry>
             <xacro:material_yaskawa_blue/>
@@ -65,5 +65,5 @@
         <collision>
             <geometry>
-                <mesh filename="package://motoman_gp280_support/meshes/gp280/collision/link_4_r.stl"/>
+                <mesh filename="package://motoman_gp250_support/meshes/gp250/collision/link_4_r.stl"/>
             </geometry>
         </collision>
@@ -72,5 +72,5 @@
         <visual>
             <geometry>
-                <mesh filename="package://motoman_gp280_support/meshes/gp280/visual/link_5_b.stl"/>
+                <mesh filename="package://motoman_gp250_support/meshes/gp250/visual/link_5_b.stl"/>
             </geometry>
             <xacro:material_yaskawa_blue/>
@@ -78,5 +78,5 @@
         <collision>
             <geometry>
-                <mesh filename="package://motoman_gp280_support/meshes/gp280/collision/link_5_b.stl"/>
+                <mesh filename="package://motoman_gp250_support/meshes/gp250/collision/link_5_b.stl"/>
             </geometry>
         </collision>
@@ -85,5 +85,5 @@
         <visual>
             <geometry>
-                <mesh filename="package://motoman_gp280_support/meshes/gp280/visual/link_6_t.stl"/>
+                <mesh filename="package://motoman_gp250_support/meshes/gp250/visual/link_6_t.stl"/>
             </geometry>
             <xacro:material_yaskawa_blue/>
@@ -91,5 +91,5 @@
         <collision>
             <geometry>
-                <mesh filename="package://motoman_gp280_support/meshes/gp280/collision/link_6_t.stl"/>
+                <mesh filename="package://motoman_gp250_support/meshes/gp250/collision/link_6_t.stl"/>
             </geometry>
         </collision>
@@ -129,5 +129,5 @@
         <parent link="${prefix}link_4_r"/>
         <child link="${prefix}link_5_b"/>
-        <origin xyz="1.015 0 0" rpy="0 0 0" />
+        <origin xyz="1.285 0 0" rpy="0 0 0" />
         <axis xyz="0 -1 0" />
         <limit lower="${radians(-125)}" upper="${radians(125)}" effort="794" velocity="${radians(250)}"/>

File: yaskawa_ros2_control_support/urdf/common_yaskawa.xacro (robot description, xacro)
@@ -25,6 +25,6 @@
     description_package="$(arg description_package)"
   />
-  <xacro:if value="${description_package == 'motoman_gp280_support'}">
-    <xacro:motoman_gp280 prefix="$(arg prefix)"/>
+  <xacro:if value="${description_package == 'motoman_gp250_support'}">
+    <xacro:motoman_gp250 prefix="$(arg prefix)"/>
   </xacro:if>
 </robot>

Commit message: modify all yamls and xacros to use the group_1 or prefix namespace

File: motoman_gp250_support/urdf/gp250_macro.xacro (robot description, xacro)
@@ -4,5 +4,5 @@
     <xacro:include filename="$(find motoman_resources)/urdf/common_materials.xacro"/>
     <!-- link list -->
-    <link name="${prefix}base_link">
+    <link name="base_link">
         <visual>
             <geometry>
@@ -98,6 +98,6 @@
     <!-- end of link list -->
     <!-- joint list -->
-    <joint name="${prefix}joint_1_s" type="revolute">
-        <parent link="${prefix}base_link"/>
+    <joint name="${prefix}joint_1" type="revolute">
+        <parent link="base_link"/>
         <child link="${prefix}link_1_s"/>
         <origin xyz="0 0 0.650" rpy="0 0 0" />
@@ -105,5 +105,5 @@
         <limit lower="${radians(-180)}" upper="${radians(180)}" effort="5516" velocity="${radians(180)}"/>
     </joint>
-    <joint name="${prefix}joint_2_l" type="revolute">
+    <joint name="${prefix}joint_2" type="revolute">
         <parent link="${prefix}link_1_s"/>
         <child link="${prefix}link_2_l"/>
@@ -112,5 +112,5 @@
         <limit lower="${radians(-60)}" upper="${radians(76)}" effort="7060" velocity="${radians(178)}"/>
     </joint>
-    <joint name="${prefix}joint_3_u" type="revolute">
+    <joint name="${prefix}joint_3" type="revolute">
         <parent link="${prefix}link_2_l"/>
         <child link="${prefix}link_3_u"/>
@@ -119,5 +119,5 @@
         <limit lower="${radians(-77.8)}" upper="${radians(197)}" effort="3089" velocity="${radians(178)}"/>
     </joint>
-    <joint name="${prefix}joint_4_r" type="revolute">
+    <joint name="${prefix}joint_4" type="revolute">
         <parent link="${prefix}link_3_u"/>
         <child link="${prefix}link_4_r"/>
@@ -126,5 +126,5 @@
         <limit lower="${radians(-360)}" upper="${radians(360)}" effort="926" velocity="${radians(250)}"/>
     </joint>
-    <joint name="${prefix}joint_5_b" type="revolute">
+    <joint name="${prefix}joint_5" type="revolute">
         <parent link="${prefix}link_4_r"/>
         <child link="${prefix}link_5_b"/>
@@ -133,5 +133,5 @@
         <limit lower="${radians(-125)}" upper="${radians(125)}" effort="794" velocity="${radians(250)}"/>
     </joint>
-    <joint name="${prefix}joint_6_t" type="revolute">
+    <joint name="${prefix}joint_6" type="revolute">
         <parent link="${prefix}link_5_b"/>
         <child link="${prefix}link_6_t"/>
@@ -140,5 +140,5 @@
         <limit lower="${radians(-360)}" upper="${radians(360)}" effort="375" velocity="${radians(360)}"/>
     </joint>
-    <joint name="${prefix}joint_6_t-tool0" type="fixed">
+    <joint name="${prefix}joint_6-tool0" type="fixed">
         <origin xyz="0.250 0 0" rpy="3.1415926 -1.570796 0"/>
         <parent link="${prefix}link_6_t"/>
@@ -147,5 +147,5 @@
     <!-- end of joint list -->
     <link name="${prefix}flange" />
-    <joint name="${prefix}joint_6_t-flange" type="fixed">
+    <joint name="${prefix}joint_6-flange" type="fixed">
         <origin xyz="0 0 0" rpy="0 ${radians(90)} 0" />
         <parent link="${prefix}link_6_t" />
@@ -156,5 +156,5 @@
     <joint name="${prefix}base_link-base" type="fixed">
         <origin xyz="0 0 0.650" rpy="0 0 0"/>
-        <parent link="${prefix}base_link"/>
+        <parent link="base_link"/>
         <child link="${prefix}base"/>
     </joint>

File: yaskawa_common_moveit/srdf/common_yaskawa.srdf.xacro (robot description, xacro)
@@ -12,19 +12,19 @@
     <!--CHAINS- When a chain is specified, all the links along the chain (including endpoints) are included in the group. Additionally, all the joints that are parents to included links are also included. This means that joints along the chain and the parent joint of the base link are included in the group-->
     <!--SUBGROUPS- Groups can also be formed by referencing to already defined group names-->
-    <group name="$(arg prefix)manipulator">
-        <chain base_link="$(arg prefix)base_link" tip_link="$(arg prefix)tool0"/>
+    <group name="manipulator">
+        <chain base_link="base_link" tip_link="$(arg prefix)tool0"/>
     </group>
-    <group_state name="home" group="$(arg prefix)manipulator">
-        <joint name="$(arg prefix)joint_1_s" value="0"/>
-        <joint name="$(arg prefix)joint_2_l" value="-1.57"/>
-        <joint name="$(arg prefix)joint_3_u" value="1.57"/>
-        <joint name="$(arg prefix)joint_4_r" value="0"/>
-        <joint name="$(arg prefix)joint_5_b" value="1.57"/>
-        <joint name="$(arg prefix)joint_6_t" value="0"/>
+    <group_state name="home" group="manipulator">
+        <joint name="$(arg prefix)joint_1" value="0"/>
+        <joint name="$(arg prefix)joint_2" value="-1.57"/>
+        <joint name="$(arg prefix)joint_3" value="1.57"/>
+        <joint name="$(arg prefix)joint_4" value="0"/>
+        <joint name="$(arg prefix)joint_5" value="1.57"/>
+        <joint name="$(arg prefix)joint_6" value="0"/>
     </group_state>
     <!--DISABLE COLLISIONS- By default it is assumed that any link of the robot could potentially come into collision with any other link in the robot. This tag disables collision checking between a specified pair of links. -->
-    <disable_collisions link1="$(arg prefix)base_link" link2="$(arg prefix)link_1_s" reason="Adjacent"/>
-    <disable_collisions link1="$(arg prefix)base_link" link2="$(arg prefix)link_2_l" reason="Never"/>
-    <disable_collisions link1="$(arg prefix)base_link" link2="$(arg prefix)link_3_u" reason="Never"/>
+    <disable_collisions link1="base_link" link2="$(arg prefix)link_1_s" reason="Adjacent"/>
+    <disable_collisions link1="base_link" link2="$(arg prefix)link_2_l" reason="Never"/>
+    <disable_collisions link1="base_link" link2="$(arg prefix)link_3_u" reason="Never"/>
     <disable_collisions link1="$(arg prefix)link_1_s" link2="$(arg prefix)link_2_l" reason="Adjacent"/>
     <disable_collisions link1="$(arg prefix)link_1_s" link2="$(arg prefix)link_3_u" reason="Never"/>

File: yaskawa_ros2_control_support/urdf/common_macro.ros2_control.xacro (robot description, xacro)
@@ -22,5 +22,5 @@
         </xacro:if>
       </hardware>
-    <joint name="${prefix}joint_1_s">
+    <joint name="${prefix}joint_1">
         <command_interface name="position">
           <param name="min">-1</param>
@@ -31,5 +31,5 @@
         </state_interface>
       </joint>
-      <joint name="${prefix}joint_2_l">
+      <joint name="${prefix}joint_2">
         <command_interface name="position">
           <param name="min">-1</param>
@@ -40,5 +40,5 @@
         </state_interface>
 	  </joint>
-      <joint name="${prefix}joint_3_u">
+      <joint name="${prefix}joint_3">
         <command_interface name="position">
           <param name="min">-1</param>
@@ -49,5 +49,5 @@
         </state_interface>
 	  </joint>
-      <joint name="${prefix}joint_4_r">
+      <joint name="${prefix}joint_4">
         <command_interface name="position">
           <param name="min">-1</param>
@@ -58,5 +58,5 @@
         </state_interface>
       </joint>
-      <joint name="${prefix}joint_5_b">
+      <joint name="${prefix}joint_5">
         <command_interface name="position">
           <param name="min">-1</param>
@@ -67,5 +67,5 @@
         </state_interface>
       </joint>
-      <joint name="${prefix}joint_6_t">
+      <joint name="${prefix}joint_6">
         <command_interface name="position">
           <param name="min">-1</param>

Commit message: added visual mesh .stl files and an rviz configuration

File: motoman_gp250_support/urdf/gp250_macro.xacro (robot description, xacro)
@@ -7,5 +7,5 @@
         <visual>
             <geometry>
-                <mesh filename="package://motoman_gp250_support/meshes/gp250/visual/base_link.stl"/>
+                <mesh filename="package://motoman_gp250_support/meshes/gp250/visual/base_link_visual.stl"/>
             </geometry>
             <xacro:material_yaskawa_blue/>
@@ -20,5 +20,5 @@
         <visual>
             <geometry>
-                <mesh filename="package://motoman_gp250_support/meshes/gp250/visual/link_1_s.stl"/>
+                <mesh filename="package://motoman_gp250_support/meshes/gp250/visual/link_1_s_visual.stl"/>
             </geometry>
             <xacro:material_yaskawa_blue/>
@@ -33,5 +33,5 @@
         <visual>
             <geometry>
-                <mesh filename="package://motoman_gp250_support/meshes/gp250/visual/link_2_l.stl"/>
+                <mesh filename="package://motoman_gp250_support/meshes/gp250/visual/link_2_l_visual.stl"/>
             </geometry>
             <xacro:material_yaskawa_blue/>
@@ -46,5 +46,5 @@
         <visual>
             <geometry>
-                <mesh filename="package://motoman_gp250_support/meshes/gp250/visual/link_3_u.stl"/>
+                <mesh filename="package://motoman_gp250_support/meshes/gp250/visual/link_3_u_visual.stl"/>
             </geometry>
             <xacro:material_yaskawa_blue/>
@@ -59,5 +59,5 @@
         <visual>
             <geometry>
-                <mesh filename="package://motoman_gp250_support/meshes/gp250/visual/link_4_r.stl"/>
+                <mesh filename="package://motoman_gp250_support/meshes/gp250/visual/link_4_r_visual.stl"/>
             </geometry>
             <xacro:material_yaskawa_blue/>
@@ -72,5 +72,5 @@
         <visual>
             <geometry>
-                <mesh filename="package://motoman_gp250_support/meshes/gp250/visual/link_5_b.stl"/>
+                <mesh filename="package://motoman_gp250_support/meshes/gp250/visual/link_5_b_visual.stl"/>
             </geometry>
             <xacro:material_yaskawa_blue/>
@@ -85,5 +85,5 @@
         <visual>
             <geometry>
-                <mesh filename="package://motoman_gp250_support/meshes/gp250/visual/link_6_t.stl"/>
+                <mesh filename="package://motoman_gp250_support/meshes/gp250/visual/link_6_t_visual.stl"/>
             </geometry>
             <xacro:material_yaskawa_blue/>

Commit message: added collision meshes for gp250

File: motoman_gp250_support/urdf/gp250_macro.xacro (robot description, xacro)
@@ -13,5 +13,5 @@
         <collision>
             <geometry>
-                <mesh filename="package://motoman_gp250_support/meshes/gp250/collision/base_link.stl"/>
+                <mesh filename="package://motoman_gp250_support/meshes/gp250/collision/base_link_collision.stl"/>
             </geometry>
         </collision>
@@ -26,5 +26,5 @@
         <collision>
             <geometry>
-                <mesh filename="package://motoman_gp250_support/meshes/gp250/collision/link_1_s.stl"/>
+                <mesh filename="package://motoman_gp250_support/meshes/gp250/collision/link_1_s_collision.stl"/>
             </geometry>
         </collision>
@@ -39,5 +39,5 @@
         <collision>
             <geometry>
-                <mesh filename="package://motoman_gp250_support/meshes/gp250/collision/link_2_l.stl"/>
+                <mesh filename="package://motoman_gp250_support/meshes/gp250/collision/link_2_l_no_balancer_collision.stl"/>
             </geometry>
         </collision>
@@ -52,5 +52,5 @@
         <collision>
             <geometry>
-                <mesh filename="package://motoman_gp250_support/meshes/gp250/collision/link_3_u.stl"/>
+                <mesh filename="package://motoman_gp250_support/meshes/gp250/collision/link_3_u_collision.stl"/>
             </geometry>
         </collision>
@@ -65,5 +65,5 @@
         <collision>
             <geometry>
-                <mesh filename="package://motoman_gp250_support/meshes/gp250/collision/link_4_r.stl"/>
+                <mesh filename="package://motoman_gp250_support/meshes/gp250/collision/link_4_r_collision.stl"/>
             </geometry>
         </collision>
@@ -78,5 +78,5 @@
         <collision>
             <geometry>
-                <mesh filename="package://motoman_gp250_support/meshes/gp250/collision/link_5_b.stl"/>
+                <mesh filename="package://motoman_gp250_support/meshes/gp250/collision/link_5_b_collision.stl"/>
             </geometry>
         </collision>
@@ -91,5 +91,5 @@
         <collision>
             <geometry>
-                <mesh filename="package://motoman_gp250_support/meshes/gp250/collision/link_6_t.stl"/>
+                <mesh filename="package://motoman_gp250_support/meshes/gp250/collision/link_6_t_collision.stl"/>
             </geometry>
         </collision>

Commit message: Add mesh files for GP 250 and GP 280 (#3)
Co-authored-by: Nikola Banović <nibanovic@gmail.com>

File: motoman_gp250_support/urdf/gp250_macro.xacro (robot description, xacro)
@@ -7,5 +7,5 @@
         <visual>
             <geometry>
-                <mesh filename="package://motoman_gp250_support/meshes/gp250/visual/base_link.stl"/>
+                <mesh filename="package://motoman_gp250_support/meshes/gp250/visual/base_link_visual.stl"/>
             </geometry>
             <xacro:material_yaskawa_blue/>
@@ -13,5 +13,5 @@
         <collision>
             <geometry>
-                <mesh filename="package://motoman_gp250_support/meshes/gp250/collision/base_link.stl"/>
+                <mesh filename="package://motoman_gp250_support/meshes/gp250/collision/base_link_collision.stl"/>
             </geometry>
         </collision>
@@ -20,5 +20,5 @@
         <visual>
             <geometry>
-                <mesh filename="package://motoman_gp250_support/meshes/gp250/visual/link_1_s.stl"/>
+                <mesh filename="package://motoman_gp250_support/meshes/gp250/visual/link_1_s_visual.stl"/>
             </geometry>
             <xacro:material_yaskawa_blue/>
@@ -26,5 +26,5 @@
         <collision>
             <geometry>
-                <mesh filename="package://motoman_gp250_support/meshes/gp250/collision/link_1_s.stl"/>
+                <mesh filename="package://motoman_gp250_support/meshes/gp250/collision/link_1_s_collision.stl"/>
             </geometry>
         </collision>
@@ -33,5 +33,5 @@
         <visual>
             <geometry>
-                <mesh filename="package://motoman_gp250_support/meshes/gp250/visual/link_2_l.stl"/>
+                <mesh filename="package://motoman_gp250_support/meshes/gp250/visual/link_2_l_visual.stl"/>
             </geometry>
             <xacro:material_yaskawa_blue/>
@@ -39,5 +39,5 @@
         <collision>
             <geometry>
-                <mesh filename="package://motoman_gp250_support/meshes/gp250/collision/link_2_l.stl"/>
+                <mesh filename="package://motoman_gp250_support/meshes/gp250/collision/link_2_l_no_balancer_collision.stl"/>
             </geometry>
         </collision>
@@ -46,5 +46,5 @@
         <visual>
             <geometry>
-                <mesh filename="package://motoman_gp250_support/meshes/gp250/visual/link_3_u.stl"/>
+                <mesh filename="package://motoman_gp250_support/meshes/gp250/visual/link_3_u_visual.stl"/>
             </geometry>
             <xacro:material_yaskawa_blue/>
@@ -52,5 +52,5 @@
         <collision>
             <geometry>
-                <mesh filename="package://motoman_gp250_support/meshes/gp250/collision/link_3_u.stl"/>
+                <mesh filename="package://motoman_gp250_support/meshes/gp250/collision/link_3_u_collision.stl"/>
             </geometry>
         </collision>
@@ -59,5 +59,5 @@
         <visual>
             <geometry>
-                <mesh filename="package://motoman_gp250_support/meshes/gp250/visual/link_4_r.stl"/>
+                <mesh filename="package://motoman_gp250_support/meshes/gp250/visual/link_4_r_visual.stl"/>
             </geometry>
             <xacro:material_yaskawa_blue/>
@@ -65,5 +65,5 @@
         <collision>
             <geometry>
-                <mesh filename="package://motoman_gp250_support/meshes/gp250/collision/link_4_r.stl"/>
+                <mesh filename="package://motoman_gp250_support/meshes/gp250/collision/link_4_r_collision.stl"/>
             </geometry>
         </collision>
@@ -72,5 +72,5 @@
         <visual>
             <geometry>
-                <mesh filename="package://motoman_gp250_support/meshes/gp250/visual/link_5_b.stl"/>
+                <mesh filename="package://motoman_gp250_support/meshes/gp250/visual/link_5_b_visual.stl"/>
             </geometry>
             <xacro:material_yaskawa_blue/>
@@ -78,5 +78,5 @@
         <collision>
             <geometry>
-                <mesh filename="package://motoman_gp250_support/meshes/gp250/collision/link_5_b.stl"/>
+                <mesh filename="package://motoman_gp250_support/meshes/gp250/collision/link_5_b_collision.stl"/>
             </geometry>
         </collision>
@@ -85,5 +85,5 @@
         <visual>
             <geometry>
-                <mesh filename="package://motoman_gp250_support/meshes/gp250/visual/link_6_t.stl"/>
+                <mesh filename="package://motoman_gp250_support/meshes/gp250/visual/link_6_t_visual.stl"/>
             </geometry>
             <xacro:material_yaskawa_blue/>
@@ -91,5 +91,5 @@
         <collision>
             <geometry>
-                <mesh filename="package://motoman_gp250_support/meshes/gp250/collision/link_6_t.stl"/>
+                <mesh filename="package://motoman_gp250_support/meshes/gp250/collision/link_6_t_collision.stl"/>
             </geometry>
         </collision>
