Commit message: Add position limits for certian scenarions. Add Yaskawa-style world frame.

File: motoman_gp250_support/urdf/gp250_macro.xacro (robot description, xacro)
@@ -1,5 +1,5 @@
 <?xml version="1.0" ?>
 <robot xmlns:xacro="http://ros.org/wiki/xacro">
-  <xacro:macro name="motoman_gp250" params="prefix">
+  <xacro:macro name="motoman_gp250" params="prefix robot_tf_frame_prefix:=r1/">
     <xacro:include filename="$(find motoman_resources)/urdf/common_materials.xacro"/>
     <!-- link list -->
@@ -159,4 +159,11 @@
         <child link="${prefix}base"/>
     </joint>
+    <!-- Motoman world frame published from the robot is the same as the base -->
+    <link name="${robot_tf_frame_prefix}world" />
+    <joint name="${prefix}base_${robot_tf_frame_prefix}world" type="fixed">
+        <origin xyz="0 0 0.0" rpy="0 0 0"/>
+        <parent link="${prefix}base"/>
+        <child link="${robot_tf_frame_prefix}world"/>
+    </joint>
   </xacro:macro>
 </robot>

Commit message: updated the gp250 URDF to run with ros2_control

File: motoman_gp250_support/urdf/gp250_macro.xacro (robot description, xacro)
@@ -1,8 +1,8 @@
 <?xml version="1.0" ?>
 <robot xmlns:xacro="http://ros.org/wiki/xacro">
-  <xacro:macro name="motoman_gp250" params="prefix">
+  <xacro:macro name="motoman_gp250" params="prefix robot_tf_frame_prefix:=r1/">
     <xacro:include filename="$(find motoman_resources)/urdf/common_materials.xacro"/>
     <!-- link list -->
-    <link name="base_link">
+    <link name="${prefix}base_link">
         <visual>
             <geometry>
@@ -17,5 +17,5 @@
         </collision>
     </link>
-    <link name="${prefix}link_1_s">
+    <link name="${prefix}link_1">
         <visual>
             <geometry>
@@ -30,5 +30,5 @@
         </collision>
     </link>
-    <link name="${prefix}link_2_l">
+    <link name="${prefix}link_2">
         <visual>
             <geometry>
@@ -43,5 +43,5 @@
         </collision>
     </link>
-    <link name="${prefix}link_3_u">
+    <link name="${prefix}link_3">
         <visual>
             <geometry>
@@ -56,5 +56,5 @@
         </collision>
     </link>
-    <link name="${prefix}link_4_r">
+    <link name="${prefix}link_4">
         <visual>
             <geometry>
@@ -69,5 +69,5 @@
         </collision>
     </link>
-    <link name="${prefix}link_5_b">
+    <link name="${prefix}link_5">
         <visual>
             <geometry>
@@ -82,5 +82,5 @@
         </collision>
     </link>
-    <link name="${prefix}link_6_t">
+    <link name="${prefix}link_6">
         <visual>
             <geometry>
@@ -98,56 +98,56 @@
     <!-- end of link list -->
     <!-- joint list -->
-    <joint name="${prefix}joint_1" type="revolute">
-        <parent link="base_link"/>
-        <child link="${prefix}link_1_s"/>
+    <joint name="${prefix}joint_s" type="revolute">
+        <parent link="${prefix}base_link"/>
+        <child link="${prefix}link_1"/>
         <origin xyz="0 0 0.650" rpy="0 0 0" />
         <axis xyz="0 0 1" />
         <limit lower="${radians(-180)}" upper="${radians(180)}" effort="5516" velocity="${radians(180)}"/>
     </joint>
-    <joint name="${prefix}joint_2" type="revolute">
-        <parent link="${prefix}link_1_s"/>
-        <child link="${prefix}link_2_l"/>
+    <joint name="${prefix}joint_l" type="revolute">
+        <parent link="${prefix}link_1"/>
+        <child link="${prefix}link_2"/>
         <origin xyz="0.285 0 0" rpy="0 0 0" />
         <axis xyz="0 1 0" />
         <limit lower="${radians(-60)}" upper="${radians(76)}" effort="7060" velocity="${radians(178)}"/>
     </joint>
-    <joint name="${prefix}joint_3" type="revolute">
-        <parent link="${prefix}link_2_l"/>
-        <child link="${prefix}link_3_u"/>
+    <joint name="${prefix}joint_u" type="revolute">
+        <parent link="${prefix}link_2"/>
+        <child link="${prefix}link_3"/>
         <origin xyz="0 0 1.150" rpy="0 0 0" />
         <axis xyz="0 -1 0" />
         <limit lower="${radians(-77.8)}" upper="${radians(197)}" effort="3089" velocity="${radians(178)}"/>
     </joint>
-    <joint name="${prefix}joint_4" type="revolute">
-        <parent link="${prefix}link_3_u"/>
-        <child link="${prefix}link_4_r"/>
+    <joint name="${prefix}joint_r" type="revolute">
+        <parent link="${prefix}link_3"/>
+        <child link="${prefix}link_4"/>
         <origin xyz="0 0 0.250" rpy="0 0 0" />
         <axis xyz="-1 0 0" />
         <limit lower="${radians(-360)}" upper="${radians(360)}" effort="926" velocity="${radians(250)}"/>
     </joint>
-    <joint name="${prefix}joint_5" type="revolute">
-        <parent link="${prefix}link_4_r"/>
-        <child link="${prefix}link_5_b"/>
+    <joint name="${prefix}joint_b" type="revolute">
+        <parent link="${prefix}link_4"/>
+        <child link="${prefix}link_5"/>
         <origin xyz="1.285 0 0" rpy="0 0 0" />
         <axis xyz="0 -1 0" />
         <limit lower="${radians(-125)}" upper="${radians(125)}" effort="794" velocity="${radians(250)}"/>
     </joint>
-    <joint name="${prefix}joint_6" type="revolute">
-        <parent link="${prefix}link_5_b"/>
-        <child link="${prefix}link_6_t"/>
+    <joint name="${prefix}joint_t" type="revolute">
+        <parent link="${prefix}link_5"/>
+        <child link="${prefix}link_6"/>
         <origin xyz="0 0 0" rpy="0 0 0" />
         <axis xyz="-1 0 0" />
         <limit lower="${radians(-360)}" upper="${radians(360)}" effort="375" velocity="${radians(360)}"/>
     </joint>
-    <joint name="${prefix}joint_6-tool0" type="fixed">
+    <joint name="${prefix}joint_t-tool0" type="fixed">
         <origin xyz="0.250 0 0" rpy="3.1415926 -1.570796 0"/>
-        <parent link="${prefix}link_6_t"/>
+        <parent link="${prefix}link_6"/>
         <child link="${prefix}tool0"/>
     </joint>
     <!-- end of joint list -->
     <link name="${prefix}flange" />
-    <joint name="${prefix}joint_6-flange" type="fixed">
+    <joint name="${prefix}joint_t-flange" type="fixed">
         <origin xyz="0 0 0" rpy="0 ${radians(90)} 0" />
-        <parent link="${prefix}link_6_t" />
+        <parent link="${prefix}link_6" />
         <child link="${prefix}flange" />
     </joint>
@@ -156,6 +156,13 @@
     <joint name="${prefix}base_link-base" type="fixed">
         <origin xyz="0 0 0.650" rpy="0 0 0"/>
-        <parent link="base_link"/>
+        <parent link="${prefix}base_link"/>
         <child link="${prefix}base"/>
+    </joint>
+    <!-- Motoman world frame published from the robot is the same as the base -->
+    <link name="${robot_tf_frame_prefix}world" />
+    <joint name="${prefix}base_${robot_tf_frame_prefix}world" type="fixed">
+        <origin xyz="0 0 0.0" rpy="0 0 0"/>
+        <parent link="${prefix}base"/>
+        <child link="${robot_tf_frame_prefix}world"/>
     </joint>
   </xacro:macro>
