Commit message: make robot work in latest gz harmonic

File: motoman_hc20_support/urdf/hc20_macro.xacro (robot description, xacro)
@@ -5,4 +5,5 @@
     <!-- link list -->
     <link name="${prefix}base_link">
+      <xacro:default_inertial/>
       <visual>
         <geometry>
@@ -18,4 +19,5 @@
     </link>
     <link name="${prefix}link_1_s">
+      <xacro:default_inertial/>
       <visual>
         <geometry>
@@ -31,4 +33,5 @@
     </link>
     <link name="${prefix}link_2_l">
+      <xacro:default_inertial/>
       <visual>
         <geometry>
@@ -44,4 +47,5 @@
     </link>
     <link name="${prefix}link_3_u">
+      <xacro:default_inertial/>
       <visual>
         <geometry>
@@ -57,4 +61,5 @@
     </link>
     <link name="${prefix}link_4_r">
+      <xacro:default_inertial/>
       <visual>
         <geometry>
@@ -70,4 +75,5 @@
     </link>
     <link name="${prefix}link_5_b">
+      <xacro:default_inertial/>
       <visual>
         <geometry>
@@ -83,4 +89,5 @@
     </link>
     <link name="${prefix}link_6_t">
+      <xacro:default_inertial/>
       <visual>
         <geometry>
@@ -95,5 +102,7 @@
       </collision>
     </link>
-    <link name="${prefix}tool0"/>
+    <link name="${prefix}tool0">
+      <xacro:default_inertial/>
+    </link>
     <!-- end of link list -->
     <!-- joint list -->
@@ -147,5 +156,7 @@
     <!-- end of joint list -->
     <!-- ROS base_link to Robot Manufacturer World Coordinates transform -->
-    <link name="${prefix}base" />
+    <link name="${prefix}base" >
+      <xacro:default_inertial/>
+    </link>
     <joint name="${prefix}base_link-base" type="fixed">
       <origin xyz="0 0 0.380" rpy="0 0 0"/>

File: motoman_ros2_control_support/urdf/common_macro.ros2_control.xacro (robot description, xacro)
@@ -95,5 +95,5 @@
       </gazebo>
       <gazebo>
-        <plugin filename="libign_ros2_control-system.so" name="ign_ros2_control::IgnitionROS2ControlPlugin">
+        <plugin filename="gz_ros2_control-system" name="gz_ros2_control::GazeboSimROS2ControlPlugin">
           <parameters>${simulation_controllers}</parameters>
           <controller_manager_node_name>${prefix}controller_manager</controller_manager_node_name>
