Commit message: fix joint orientation

File: motoman_hc20_support/urdf/hc20sdtp_macro.xacro (robot description, xacro)
@@ -1,5 +1,5 @@
 <?xml version="1.0" ?>
 <robot xmlns:xacro="http://ros.org/wiki/xacro">
-  <xacro:macro name="motoman_hc20sdtp" params="prefix">
+  <xacro:macro name="motoman_hc20sdtp" params="prefix robot_tf_frame_prefix:=r1/">
     <xacro:include filename="$(find motoman_resources)/urdf/common_materials.xacro"/>
     <!-- link list -->
@@ -7,5 +7,6 @@
       <visual>
         <geometry>
-          <mesh filename="package://motoman_hc10_support/meshes/hc10/visual/base_link.dae"/>
+          <!-- <mesh filename="package://motoman_hc10_support/meshes/hc10/visual/base_link.dae"/> -->
+          <mesh filename="package://motoman_hc20_support/meshes/hc20/visual/base_link.stl" scale="0.923 0.923 0.923"/>
         </geometry>
         <xacro:material_yaskawa_blue/>
@@ -13,5 +14,6 @@
       <collision>
         <geometry>
-          <mesh filename="package://motoman_hc10_support/meshes/hc10/collision/base_link.stl"/>
+          <!-- <mesh filename="package://motoman_hc10_support/meshes/hc10/collision/base_link.stl"/> -->
+          <mesh filename="package://motoman_hc20_support/meshes/hc20/collision/base_link.stl" scale="0.923 0.923 0.923"/>
         </geometry>
       </collision>
@@ -20,5 +22,6 @@
       <visual>
         <geometry>
-          <mesh filename="package://motoman_hc10_support/meshes/hc10/visual/link_1_s.dae"/>
+          <!-- <mesh filename="package://motoman_hc10_support/meshes/hc10/visual/link_1_s.dae"/> -->
+          <mesh filename="package://motoman_hc20_support/meshes/hc20/visual/link_1_s.stl" scale="0.9 0.9 0.9"/>
         </geometry>
         <xacro:material_yaskawa_blue/>
@@ -26,5 +29,6 @@
       <collision>
         <geometry>
-          <mesh filename="package://motoman_hc10_support/meshes/hc10/collision/link_1_s.stl"/>
+          <!-- <mesh filename="package://motoman_hc10_support/meshes/hc10/collision/link_1_s.stl"/> -->
+          <mesh filename="package://motoman_hc20_support/meshes/hc20/collision/link_1_s.stl" scale="0.9 0.9 0.9"/>
         </geometry>
       </collision>
@@ -33,5 +37,5 @@
       <visual>
         <geometry>
-          <mesh filename="package://motoman_hc10_support/meshes/hc10/visual/link_2_l.dae"/>
+          <mesh filename="package://motoman_hc10_support/meshes/hc10/visual/link_2_l.dae" scale="1.0357 1.0357 1.0357"/>
         </geometry>
         <xacro:material_yaskawa_blue/>
@@ -39,5 +43,5 @@
       <collision>
         <geometry>
-          <mesh filename="package://motoman_hc10_support/meshes/hc10/collision/link_2_l.stl"/>
+          <mesh filename="package://motoman_hc10_support/meshes/hc10/collision/link_2_l.stl" scale="1.0357 1.0357 1.0357"/>
         </geometry>
       </collision>
@@ -46,5 +50,6 @@
       <visual>
         <geometry>
-          <mesh filename="package://motoman_hc10_support/meshes/hc10/visual/link_3_u.dae"/>
+          <mesh filename="package://motoman_hc10_support/meshes/hc10/visual/link_3_u.dae" scale="1.2 1.2 1.2"/>
+          <!-- <mesh filename="package://motoman_hc20_support/meshes/hc20/visual/link_3_u.stl"/> -->
         </geometry>
         <xacro:material_yaskawa_blue/>
@@ -52,5 +57,6 @@
       <collision>
         <geometry>
-          <mesh filename="package://motoman_hc10_support/meshes/hc10/collision/link_3_u.stl"/>
+          <mesh filename="package://motoman_hc10_support/meshes/hc10/collision/link_3_u.stl" scale="1.2 1.2 1.2"/>
+          <!-- <mesh filename="package://motoman_hc20_support/meshes/hc20/collision/link_3_u.stl"/> -->
         </geometry>
       </collision>
@@ -115,5 +121,5 @@
       <parent link="${prefix}link_2_l"/>
       <child link="${prefix}link_3_u"/>
-      <origin xyz="0 0 0.725" rpy="0 0 0" />
+      <origin xyz="0 0 0.725" rpy="0 -1.57 0" />
       <axis xyz="0 -1 0" />
       <limit lower="${radians(-290)}" upper="${radians(290)}" effort="141.12" velocity="${radians(135)}"/>
@@ -136,5 +142,5 @@
       <parent link="${prefix}link_5_b"/>
       <child link="${prefix}link_6_t"/>
-      <origin xyz="0 0 0" rpy="0 0 0" />
+      <origin xyz="0 0 0" rpy="0 0 1.57" />
       <axis xyz="0 0 1" />
       <limit lower="${radians(-210)}" upper="${radians(210)}" effort="29.4" velocity="${radians(180)}"/>
@@ -146,4 +152,10 @@
     </joint>
     <!-- end of joint list -->
+    <link name="${prefix}flange" />
+    <joint name="${prefix}joint_6_t-flange" type="fixed">
+        <origin xyz="0 0 0" rpy="0 ${radians(90)} 0" />
+        <parent link="${prefix}link_6_t" />
+        <child link="${prefix}flange" />
+    </joint>
     <!-- ROS base_link to Robot Manufacturer World Coordinates transform -->
     <link name="${prefix}base" />
@@ -153,4 +165,11 @@
       <child link="${prefix}base"/>
     </joint>
+    <!-- Motoman world frame published from the robot is the same as the base -->
+    <link name="${robot_tf_frame_prefix}world" />
+    <joint name="${prefix}base_${robot_tf_frame_prefix}world" type="fixed">
+        <origin xyz="0 0 0.0" rpy="0 0 0"/>
+        <parent link="${prefix}base"/>
+        <child link="${robot_tf_frame_prefix}world"/>
+    </joint>
   </xacro:macro>
 </robot>

Commit message: update hc20stdp meshes

File: motoman_hc20_support/urdf/hc20sdtp_macro.xacro (robot description, xacro)
@@ -7,5 +7,5 @@
       <visual>
         <geometry>
-          <mesh filename="package://motoman_hc10_support/meshes/hc10/visual/base_link.dae"/>
+          <mesh filename="package://motoman_hc20_support/meshes/hc20sdtp/visual/base_link.dae"/>
         </geometry>
         <xacro:material_yaskawa_blue/>
@@ -13,5 +13,5 @@
       <collision>
         <geometry>
-          <mesh filename="package://motoman_hc10_support/meshes/hc10/collision/base_link.stl"/>
+          <mesh filename="package://motoman_hc20_support/meshes/hc20sdtp/collision/base_link.stl"/>
         </geometry>
       </collision>
@@ -20,5 +20,5 @@
       <visual>
         <geometry>
-          <mesh filename="package://motoman_hc10_support/meshes/hc10/visual/link_1_s.dae"/>
+          <mesh filename="package://motoman_hc20_support/meshes/hc20sdtp/visual/link_1_s.dae"/>
         </geometry>
         <xacro:material_yaskawa_blue/>
@@ -26,5 +26,5 @@
       <collision>
         <geometry>
-          <mesh filename="package://motoman_hc10_support/meshes/hc10/collision/link_1_s.stl"/>
+          <mesh filename="package://motoman_hc20_support/meshes/hc20sdtp/collision/link_1_s.stl"/>
         </geometry>
       </collision>
@@ -33,5 +33,5 @@
       <visual>
         <geometry>
-          <mesh filename="package://motoman_hc10_support/meshes/hc10/visual/link_2_l.dae"/>
+          <mesh filename="package://motoman_hc20_support/meshes/hc20sdtp/visual/link_2_l.dae"/>
         </geometry>
         <xacro:material_yaskawa_blue/>
@@ -39,5 +39,5 @@
       <collision>
         <geometry>
-          <mesh filename="package://motoman_hc10_support/meshes/hc10/collision/link_2_l.stl"/>
+          <mesh filename="package://motoman_hc20_support/meshes/hc20sdtp/collision/link_2_l.stl"/>
         </geometry>
       </collision>
@@ -46,5 +46,5 @@
       <visual>
         <geometry>
-          <mesh filename="package://motoman_hc10_support/meshes/hc10/visual/link_3_u.dae"/>
+          <mesh filename="package://motoman_hc20_support/meshes/hc20sdtp/visual/link_3_u.dae"/>
         </geometry>
         <xacro:material_yaskawa_blue/>
@@ -52,5 +52,5 @@
       <collision>
         <geometry>
-          <mesh filename="package://motoman_hc10_support/meshes/hc10/collision/link_3_u.stl"/>
+          <mesh filename="package://motoman_hc20_support/meshes/hc20sdtp/collision/link_3_u.stl"/>
         </geometry>
       </collision>
@@ -59,5 +59,5 @@
       <visual>
         <geometry>
-          <mesh filename="package://motoman_hc10_support/meshes/hc10/visual/link_4_r.dae"/>
+          <mesh filename="package://motoman_hc20_support/meshes/hc20sdtp/visual/link_4_r.dae"/>
         </geometry>
         <xacro:material_yaskawa_blue/>
@@ -65,5 +65,5 @@
       <collision>
         <geometry>
-          <mesh filename="package://motoman_hc10_support/meshes/hc10/collision/link_4_r.stl"/>
+          <mesh filename="package://motoman_hc20_support/meshes/hc20sdtp/collision/link_4_r.stl"/>
         </geometry>
       </collision>
@@ -72,5 +72,5 @@
       <visual>
         <geometry>
-          <mesh filename="package://motoman_hc10_support/meshes/hc10/visual/link_5_b.dae"/>
+          <mesh filename="package://motoman_hc20_support/meshes/hc20sdtp/visual/link_5_b.dae"/>
         </geometry>
         <xacro:material_yaskawa_blue/>
@@ -78,5 +78,5 @@
       <collision>
         <geometry>
-          <mesh filename="package://motoman_hc10_support/meshes/hc10/collision/link_5_b.stl"/>
+          <mesh filename="package://motoman_hc20_support/meshes/hc20sdtp/collision/link_5_b.stl"/>
         </geometry>
       </collision>
@@ -85,5 +85,5 @@
       <visual>
         <geometry>
-          <mesh filename="package://motoman_hc10_support/meshes/hc10dt/visual/link_6_t.dae"/>
+          <mesh filename="package://motoman_hc20_support/meshes/hc20sdtp/visual/link_6_t.dae"/>
         </geometry>
         <xacro:material_yaskawa_blue/>
@@ -91,5 +91,5 @@
       <collision>
         <geometry>
-          <mesh filename="package://motoman_hc10_support/meshes/hc10dt/collision/link_6_t.stl"/>
+          <mesh filename="package://motoman_hc20_support/meshes/hc20sdtp/collision/link_6_t.stl"/>
        </geometry>
       </collision>
@@ -122,5 +122,5 @@
       <parent link="${prefix}link_3_u"/>
       <child link="${prefix}link_4_r"/>
-      <origin xyz="0 0 -0.475" rpy="0 0 0" />
+      <origin xyz="0.475 0 0" rpy="0 0 0" />
       <axis xyz="0 0 1" />
       <limit lower="${radians(-210)}" upper="${radians(210)}" effort="58.8" velocity="${radians(130)}"/>
@@ -136,10 +136,10 @@
       <parent link="${prefix}link_5_b"/>
       <child link="${prefix}link_6_t"/>
-      <origin xyz="0 0 0" rpy="0 0 0" />
+      <origin xyz="0.200 0 0" rpy="0 0 0" />
       <axis xyz="0 0 1" />
       <limit lower="${radians(-210)}" upper="${radians(210)}" effort="29.4" velocity="${radians(180)}"/>
     </joint>
     <joint name="${prefix}joint_6_t-tool0" type="fixed">
-      <origin xyz="0 0 -0.200" rpy="${pi} 0 0"/>
+      <origin xyz="0 0 0" rpy="${radians(180)} ${radians(-90)} 0"/>
       <parent link="${prefix}link_6_t"/>
       <child link="${prefix}tool0"/>

Commit message: adjust to hc20sdtp Co-authored-by: Nikola Banovic <nibanovic@gmail.com>

File: motoman_hc20_support/urdf/hc20sdtp_macro.xacro (robot description, xacro)
@@ -1,5 +1,5 @@
 <?xml version="1.0" ?>
 <robot xmlns:xacro="http://ros.org/wiki/xacro">
-  <xacro:macro name="motoman_hc20sdtp" params="prefix robot_tf_frame_prefix:=r1/">
+  <xacro:macro name="motoman_hc20sdtp" params="prefix robot_tf_frame_prefix:=hc20sdtp/">
     <xacro:include filename="$(find motoman_resources)/urdf/common_materials.xacro"/>
     <!-- link list -->
@@ -7,6 +7,5 @@
       <visual>
         <geometry>
-          <!-- <mesh filename="package://motoman_hc10_support/meshes/hc10/visual/base_link.dae"/> -->
-          <mesh filename="package://motoman_hc20_support/meshes/hc20/visual/base_link.stl" scale="0.923 0.923 0.923"/>
+          <mesh filename="package://motoman_hc20_support/meshes/hc20sdtp/visual/base_link.dae"/>
         </geometry>
         <xacro:material_yaskawa_blue/>
@@ -14,6 +13,5 @@
       <collision>
         <geometry>
-          <!-- <mesh filename="package://motoman_hc10_support/meshes/hc10/collision/base_link.stl"/> -->
-          <mesh filename="package://motoman_hc20_support/meshes/hc20/collision/base_link.stl" scale="0.923 0.923 0.923"/>
+          <mesh filename="package://motoman_hc20_support/meshes/hc20sdtp/collision/base_link.stl"/>
         </geometry>
       </collision>
@@ -22,6 +20,5 @@
       <visual>
         <geometry>
-          <!-- <mesh filename="package://motoman_hc10_support/meshes/hc10/visual/link_1_s.dae"/> -->
-          <mesh filename="package://motoman_hc20_support/meshes/hc20/visual/link_1_s.stl" scale="0.9 0.9 0.9"/>
+          <mesh filename="package://motoman_hc20_support/meshes/hc20sdtp/visual/link_1_s.dae"/>
         </geometry>
         <xacro:material_yaskawa_blue/>
@@ -29,6 +26,5 @@
       <collision>
         <geometry>
-          <!-- <mesh filename="package://motoman_hc10_support/meshes/hc10/collision/link_1_s.stl"/> -->
-          <mesh filename="package://motoman_hc20_support/meshes/hc20/collision/link_1_s.stl" scale="0.9 0.9 0.9"/>
+          <mesh filename="package://motoman_hc20_support/meshes/hc20sdtp/collision/link_1_s.stl"/>
         </geometry>
       </collision>
@@ -37,5 +33,5 @@
       <visual>
         <geometry>
-          <mesh filename="package://motoman_hc10_support/meshes/hc10/visual/link_2_l.dae" scale="1.0357 1.0357 1.0357"/>
+          <mesh filename="package://motoman_hc20_support/meshes/hc20sdtp/visual/link_2_l.dae"/>
         </geometry>
         <xacro:material_yaskawa_blue/>
@@ -43,5 +39,5 @@
       <collision>
         <geometry>
-          <mesh filename="package://motoman_hc10_support/meshes/hc10/collision/link_2_l.stl" scale="1.0357 1.0357 1.0357"/>
+          <mesh filename="package://motoman_hc20_support/meshes/hc20sdtp/collision/link_2_l.stl"/>
         </geometry>
       </collision>
@@ -49,14 +45,14 @@
     <link name="${prefix}link_3_u">
       <visual>
+        <origin xyz="0 0 0" rpy="0 ${radians(90)} 0"/>
         <geometry>
-          <mesh filename="package://motoman_hc10_support/meshes/hc10/visual/link_3_u.dae" scale="1.2 1.2 1.2"/>
-          <!-- <mesh filename="package://motoman_hc20_support/meshes/hc20/visual/link_3_u.stl"/> -->
+          <mesh filename="package://motoman_hc20_support/meshes/hc20sdtp/visual/link_3_u.dae"/>
         </geometry>
         <xacro:material_yaskawa_blue/>
       </visual>
       <collision>
+        <origin xyz="0 0 0" rpy="0 ${radians(90)} 0"/>
         <geometry>
-          <mesh filename="package://motoman_hc10_support/meshes/hc10/collision/link_3_u.stl" scale="1.2 1.2 1.2"/>
-          <!-- <mesh filename="package://motoman_hc20_support/meshes/hc20/collision/link_3_u.stl"/> -->
+          <mesh filename="package://motoman_hc20_support/meshes/hc20sdtp/collision/link_3_u.stl"/>
         </geometry>
       </collision>
@@ -64,12 +60,14 @@
     <link name="${prefix}link_4_r">
       <visual>
+        <origin xyz="0 0 0" rpy="0 ${radians(90)} 0"/>
         <geometry>
-          <mesh filename="package://motoman_hc10_support/meshes/hc10/visual/link_4_r.dae"/>
+          <mesh filename="package://motoman_hc20_support/meshes/hc20sdtp/visual/link_4_r.dae"/>
         </geometry>
         <xacro:material_yaskawa_blue/>
       </visual>
       <collision>
+        <origin xyz="0 0 0" rpy="0 ${radians(90)} 0"/>
         <geometry>
-          <mesh filename="package://motoman_hc10_support/meshes/hc10/collision/link_4_r.stl"/>
+          <mesh filename="package://motoman_hc20_support/meshes/hc20sdtp/collision/link_4_r.stl"/>
         </geometry>
       </collision>
@@ -77,12 +75,14 @@
     <link name="${prefix}link_5_b">
       <visual>
+        <origin xyz="0 0 0" rpy="0 ${radians(90)} 0"/>
         <geometry>
-          <mesh filename="package://motoman_hc10_support/meshes/hc10/visual/link_5_b.dae"/>
+          <mesh filename="package://motoman_hc20_support/meshes/hc20sdtp/visual/link_5_b.dae"/>
         </geometry>
         <xacro:material_yaskawa_blue/>
       </visual>
       <collision>
+        <origin xyz="0 0 0" rpy="0 ${radians(90)} 0"/>
         <geometry>
-          <mesh filename="package://motoman_hc10_support/meshes/hc10/collision/link_5_b.stl"/>
+          <mesh filename="package://motoman_hc20_support/meshes/hc20sdtp/collision/link_5_b.stl"/>
         </geometry>
       </collision>
@@ -90,12 +90,14 @@
     <link name="${prefix}link_6_t">
       <visual>
+        <origin xyz="0 0 0" rpy="0 ${radians(90)} 0"/>
         <geometry>
-          <mesh filename="package://motoman_hc10_support/meshes/hc10dt/visual/link_6_t.dae"/>
+          <mesh filename="package://motoman_hc20_support/meshes/hc20sdtp/visual/link_6_t.dae"/>
         </geometry>
         <xacro:material_yaskawa_blue/>
       </visual>
       <collision>
+        <origin xyz="0 0 0" rpy="0 ${radians(90)} 0"/>
         <geometry>
-          <mesh filename="package://motoman_hc10_support/meshes/hc10dt/collision/link_6_t.stl"/>
+          <mesh filename="package://motoman_hc20_support/meshes/hc20sdtp/collision/link_6_t.stl"/>
        </geometry>
       </collision>
@@ -142,20 +144,14 @@
       <parent link="${prefix}link_5_b"/>
       <child link="${prefix}link_6_t"/>
-      <origin xyz="0 0 0" rpy="0 0 1.57" />
+      <origin xyz="0 0 -0.200" rpy="0 0 ${radians(90)}" />
       <axis xyz="0 0 1" />
       <limit lower="${radians(-210)}" upper="${radians(210)}" effort="29.4" velocity="${radians(180)}"/>
     </joint>
     <joint name="${prefix}joint_6_t-tool0" type="fixed">
-      <origin xyz="0 0 -0.200" rpy="${pi} 0 0"/>
+      <origin xyz="0 0 0" rpy="${pi} 0 ${radians(-90)}"/>
       <parent link="${prefix}link_6_t"/>
       <child link="${prefix}tool0"/>
     </joint>
     <!-- end of joint list -->
-    <link name="${prefix}flange" />
-    <joint name="${prefix}joint_6_t-flange" type="fixed">
-        <origin xyz="0 0 0" rpy="0 ${radians(90)} 0" />
-        <parent link="${prefix}link_6_t" />
-        <child link="${prefix}flange" />
-    </joint>
     <!-- ROS base_link to Robot Manufacturer World Coordinates transform -->
     <link name="${prefix}base" />

Commit message: use radians method

File: motoman_hc20_support/urdf/hc20sdtp_macro.xacro (robot description, xacro)
@@ -123,5 +123,5 @@
       <parent link="${prefix}link_2_l"/>
       <child link="${prefix}link_3_u"/>
-      <origin xyz="0 0 0.725" rpy="0 -1.57 0" />
+      <origin xyz="0 0 0.725" rpy="0 ${radians(-90)} 0" />
       <axis xyz="0 -1 0" />
       <limit lower="${radians(-290)}" upper="${radians(290)}" effort="141.12" velocity="${radians(135)}"/>

Commit message: fix gazebo missing inertial

File: motoman_hc20_support/urdf/hc20sdtp_macro.xacro (robot description, xacro)
@@ -5,9 +5,10 @@
     <!-- link list -->
     <link name="${prefix}base_link">
+      <xacro:default_inertial/>
       <visual>
         <geometry>
           <mesh filename="package://motoman_hc20_support/meshes/hc20sdtp/visual/base_link.dae"/>
         </geometry>
-        <xacro:material_yaskawa_blue/>
+        <xacro:material_yaskawa_white/>
       </visual>
       <collision>
@@ -18,9 +19,10 @@
     </link>
     <link name="${prefix}link_1_s">
+      <xacro:default_inertial/>
       <visual>
         <geometry>
           <mesh filename="package://motoman_hc20_support/meshes/hc20sdtp/visual/link_1_s.dae"/>
         </geometry>
-        <xacro:material_yaskawa_blue/>
+        <xacro:material_yaskawa_white/>
       </visual>
       <collision>
@@ -31,9 +33,10 @@
     </link>
     <link name="${prefix}link_2_l">
+      <xacro:default_inertial/>
       <visual>
         <geometry>
           <mesh filename="package://motoman_hc20_support/meshes/hc20sdtp/visual/link_2_l.dae"/>
         </geometry>
-        <xacro:material_yaskawa_blue/>
+        <xacro:material_yaskawa_white/>
       </visual>
       <collision>
@@ -44,4 +47,5 @@
     </link>
     <link name="${prefix}link_3_u">
+      <xacro:default_inertial/>
       <visual>
         <origin xyz="0 0 0" rpy="0 ${radians(90)} 0"/>
@@ -49,5 +53,5 @@
           <mesh filename="package://motoman_hc20_support/meshes/hc20sdtp/visual/link_3_u.dae"/>
         </geometry>
-        <xacro:material_yaskawa_blue/>
+        <xacro:material_yaskawa_white/>
       </visual>
       <collision>
@@ -59,4 +63,5 @@
     </link>
     <link name="${prefix}link_4_r">
+      <xacro:default_inertial/>
       <visual>
         <origin xyz="0 0 0" rpy="0 ${radians(90)} 0"/>
@@ -64,5 +69,5 @@
           <mesh filename="package://motoman_hc20_support/meshes/hc20sdtp/visual/link_4_r.dae"/>
         </geometry>
-        <xacro:material_yaskawa_blue/>
+        <xacro:material_yaskawa_white/>
       </visual>
       <collision>
@@ -74,4 +79,5 @@
     </link>
     <link name="${prefix}link_5_b">
+      <xacro:default_inertial/>
       <visual>
         <origin xyz="0 0 0" rpy="0 ${radians(90)} 0"/>
@@ -79,5 +85,5 @@
           <mesh filename="package://motoman_hc20_support/meshes/hc20sdtp/visual/link_5_b.dae"/>
         </geometry>
-        <xacro:material_yaskawa_blue/>
+        <xacro:material_yaskawa_white/>
       </visual>
       <collision>
@@ -89,4 +95,5 @@
     </link>
     <link name="${prefix}link_6_t">
+      <xacro:default_inertial/>
       <visual>
         <origin xyz="0 0 0" rpy="0 ${radians(90)} 0"/>
@@ -94,5 +101,5 @@
           <mesh filename="package://motoman_hc20_support/meshes/hc20sdtp/visual/link_6_t.dae"/>
         </geometry>
-        <xacro:material_yaskawa_blue/>
+        <xacro:material_yaskawa_white/>
       </visual>
       <collision>
@@ -103,5 +110,7 @@
       </collision>
     </link>
-    <link name="${prefix}tool0"/>
+    <link name="${prefix}tool0">
+      <xacro:default_inertial/>
+    </link>
     <!-- end of link list -->
     <!-- joint list -->
@@ -155,5 +164,7 @@
     <!-- end of joint list -->
     <!-- ROS base_link to Robot Manufacturer World Coordinates transform -->
-    <link name="${prefix}base" />
+    <link name="${prefix}base">
+      <xacro:default_inertial/>
+    </link>
     <joint name="${prefix}base_link-base" type="fixed">
       <origin xyz="0 0 0.360" rpy="0 0 0"/>
@@ -162,5 +173,7 @@
     </joint>
     <!-- Motoman world frame published from the robot is the same as the base -->
-    <link name="${robot_tf_frame_prefix}world" />
+    <link name="${robot_tf_frame_prefix}world">
+      <xacro:default_inertial/>
+    </link>
     <joint name="${prefix}base_${robot_tf_frame_prefix}world" type="fixed">
         <origin xyz="0 0 0.0" rpy="0 0 0"/>

Commit message: fix link_6_t rotation

File: motoman_hc20_support/urdf/hc20sdtp_macro.xacro (robot description, xacro)
@@ -97,5 +97,5 @@
       <xacro:default_inertial/>
       <visual>
-        <origin xyz="0 0 0" rpy="0 ${radians(90)} 0"/>
+        <origin xyz="0 0 0" rpy="0 ${radians(90)} ${radians(-90)}"/>
         <geometry>
           <mesh filename="package://motoman_hc20_support/meshes/hc20sdtp/visual/link_6_t.dae"/>
@@ -104,5 +104,5 @@
       </visual>
       <collision>
-        <origin xyz="0 0 0" rpy="0 ${radians(90)} 0"/>
+        <origin xyz="0 0 0" rpy="0 ${radians(90)} ${radians(-90)}"/>
         <geometry>
           <mesh filename="package://motoman_hc20_support/meshes/hc20sdtp/collision/link_6_t.stl"/>
