Commit message: mh5: update joint/links to include numbers

File: motoman_mh5_support/urdf/mh5_macro.xacro (robot description, xacro)
@@ -20,5 +20,5 @@
 			</collision>
 		</link>
-		<link name="${prefix}link_s">
+		<link name="${prefix}link_1_s">
 			<visual>
 				<geometry>
@@ -34,5 +34,5 @@
 			</collision>
 		</link>
-		<link name="${prefix}link_l">
+		<link name="${prefix}link_2_l">
 			<visual>
 				<!-- <origin rpy="1.57 3.1416 0" xyz="0 0 0"/> -->
@@ -50,5 +50,5 @@
 			</collision>
 		</link>
-		<link name="${prefix}link_u">
+		<link name="${prefix}link_3_u">
 			<visual>
 				<!-- <origin rpy="1.57 -3.1415 0" xyz="0 0 0"/> -->
@@ -66,5 +66,5 @@
 			</collision>
 		</link>
-		<link name="${prefix}link_r">
+		<link name="${prefix}link_4_r">
 			<visual>
 				<!-- <origin rpy="0 0 3.1416" xyz="0 0 0"/> -->
@@ -82,5 +82,5 @@
 			</collision>
 		</link>
-		<link name="${prefix}link_b">
+		<link name="${prefix}link_5_b">
 			<visual>
 				<!-- <origin rpy="-1.57 0 3.1416" xyz="0 0 0"/> -->
@@ -98,5 +98,5 @@
 			</collision>
 		</link>
-		<link name="${prefix}link_t">
+		<link name="${prefix}link_6_t">
 			<visual>
 				<geometry>
@@ -114,47 +114,47 @@
 		<!-- end of link list -->
 		<!-- joint list -->
-		<joint name="${prefix}joint_s" type="revolute">
+		<joint name="${prefix}joint_1_s" type="revolute">
 			<parent link="${prefix}base_link"/>
-			<child link="${prefix}link_s"/>
+			<child link="${prefix}link_1_s"/>
 			<origin xyz="0 0 0.1990" rpy="0 0 0"/>
 			<axis xyz="0 0 1" />
 			<limit lower="-2.9671" upper="2.9671" effort="100" velocity="2.96" />
 		</joint>
-		<joint name="${prefix}joint_l" type="revolute">
-			<parent link="${prefix}link_s"/>
-			<child link="${prefix}link_l"/>
+		<joint name="${prefix}joint_2_l" type="revolute">
+			<parent link="${prefix}link_1_s"/>
+			<child link="${prefix}link_2_l"/>
 			<origin xyz="0.0880 0 0.1310" rpy="0 0 0"/>
 			<axis xyz="0 1 0" />
 			<limit lower="-1.1345" upper="2.6180" effort="100" velocity="2.96" />
 		</joint>
-		<joint name="${prefix}joint_u" type="revolute">
-			<parent link="${prefix}link_l"/>
-			<child link="${prefix}link_u"/>
+		<joint name="${prefix}joint_3_u" type="revolute">
+			<parent link="${prefix}link_2_l"/>
+			<child link="${prefix}link_3_u"/>
 			<origin xyz="0 0 0.3100" rpy="0 0 0"/>
 			<axis xyz="0 -1 0" />
-      <!-- Old limits: lower="-2.3736" upper="4.4506" The new limits
-           below were measured from an MH5F.  They ensure that link_r
-           won't hit link_l even when joint_r is at 45 degrees.  The
+      <!-- Old limits lower="-2.3736" upper="4.4506" The new limits
+           below were measured from an MH5F.  They ensure that link_4_r
+           won't hit link_2_l even when joint_r is at 45 degrees.  The
            old limits were converted directly from the MH5 data sheet,
            which was clearly way off. -->
 			<limit lower="-1.0122" upper="3.2218" effort="100" velocity="2.96" />
 		</joint>
-		<joint name="${prefix}joint_r" type="revolute">
-			<parent link="${prefix}link_u"/>
-			<child link="${prefix}link_r"/>
+		<joint name="${prefix}joint_4_r" type="revolute">
+			<parent link="${prefix}link_3_u"/>
+			<child link="${prefix}link_4_r"/>
 			<origin xyz="0.0715 0 0.0399" rpy="0 0 0"/>
 			<axis xyz="-1 0 0" />
 			<limit lower="-3.3161" upper="3.3161" effort="100" velocity="3.48" />
 		</joint>
-		<joint name="${prefix}joint_b" type="revolute">
-			<parent link="${prefix}link_r"/>
-			<child link="${prefix}link_b"/>
+		<joint name="${prefix}joint_5_b" type="revolute">
+			<parent link="${prefix}link_4_r"/>
+			<child link="${prefix}link_5_b"/>
 			<origin xyz="0.2335 0 0" rpy="0 0 0"/>
 			<axis xyz="0 -1 0" />
 			<limit lower="-2.1817" upper="2.1817" effort="100" velocity="3.48" />
 		</joint>
-		<joint name="${prefix}joint_t" type="revolute">
-			<parent link="${prefix}link_b"/>
-			<child link="${prefix}link_t"/>
+		<joint name="${prefix}joint_6_t" type="revolute">
+			<parent link="${prefix}link_5_b"/>
+			<child link="${prefix}link_6_t"/>
 			<origin xyz="0.0865 0 0" rpy="0 0 0"/>
 			<axis xyz="-1 0 0" />

File: motoman_ros2_control_support/urdf/common_macro.ros2_control.xacro (robot description, xacro)
@@ -5,9 +5,5 @@
                prefix
                joints_with_suffix:=^|false
-               use_mock_hardware:=^|false
-               sim_gazebo_classic:=^|false
-               sim_gazebo:=^|false
-               simulation_controllers
-               description_package"
+               use_mock_hardware:=^|false"
                >
     <xacro:property name="joint_1_suffix" value=""/>
@@ -29,10 +25,4 @@
         <xacro:if value="${use_mock_hardware}">
           <plugin>mock_components/GenericSystem</plugin>
-        </xacro:if>
-        <xacro:if value="${sim_gazebo_classic}">
-          <plugin>gazebo_ros2_control/GazeboSystem</plugin>
-        </xacro:if>
-        <xacro:if value="${sim_gazebo}">
-          <plugin>ign_ros2_control/IgnitionSystem</plugin>
         </xacro:if>
       </hardware>
@@ -80,25 +70,4 @@
       </joint>
     </ros2_control>
-    <xacro:if value="$(arg sim_gazebo_classic)">
-      <!-- Gazebo plugins -->
-      <gazebo reference="world">
-      </gazebo>
-      <gazebo>
-        <plugin filename="libgazebo_ros2_control.so" name="gazebo_ros2_control">
-          <parameters>${simulation_controllers}</parameters>
-        </plugin>
-      </gazebo>
-    </xacro:if>
-    <xacro:if value="$(arg sim_gazebo)">
-      <!-- Gazebo plugins -->
-      <gazebo reference="world">
-      </gazebo>
-      <gazebo>
-        <plugin filename="libign_ros2_control-system.so" name="ign_ros2_control::IgnitionROS2ControlPlugin">
-          <parameters>${simulation_controllers}</parameters>
-          <controller_manager_node_name>${prefix}controller_manager</controller_manager_node_name>
-        </plugin>
-      </gazebo>
-    </xacro:if>
   </xacro:macro>
 </robot>

File: motoman_ros2_control_support/urdf/common_motoman.xacro (robot description, xacro)
@@ -8,7 +8,4 @@
   <!-- ros2_control mock and simulation plugins -->
   <xacro:arg name="use_mock_hardware" default="false" />
-  <xacro:arg name="sim_gazebo_classic" default="false" />
-  <xacro:arg name="sim_gazebo" default="false" />
-  <xacro:arg name="simulation_controllers" default="" />
   <xacro:property name="description_package" value="$(arg description_package)"/>
   <xacro:property name="description_macro_file" value="$(arg description_macro_file)"/>
@@ -22,8 +19,4 @@
     joints_with_suffix="$(arg joints_with_suffix)"
     use_mock_hardware="$(arg use_mock_hardware)"
-    sim_gazebo_classic="$(arg sim_gazebo_classic)"
-    sim_gazebo="$(arg sim_gazebo)"
-    simulation_controllers="$(arg simulation_controllers)"
-    description_package="$(arg description_package)"
   />
   <xacro:if value="${description_package == 'motoman_gp250_support'}">

Commit message: rotate joint_5_b pitch 90 deg

File: motoman_mh5_support/urdf/mh5_macro.xacro (robot description, xacro)
@@ -150,5 +150,5 @@
 			<parent link="${prefix}link_4_r"/>
 			<child link="${prefix}link_5_b"/>
-			<origin xyz="0.2335 0 0" rpy="0 0 0"/>
+			<origin xyz="0.2335 0 0" rpy="0 1.571 0"/>
 			<axis xyz="0 -1 0" />
 			<limit lower="-2.1817" upper="2.1817" effort="100" velocity="3.48" />
