Commit message: Change the remaining yaskawa_ prefixes to motoman_prefixes, also inside files

File: motoman_ros2_control_support/urdf/common_macro.ros2_control.xacro (robot description, xacro)
@@ -1,5 +1,5 @@
 <?xml version="1.0"?>
 <robot xmlns:xacro="http://www.ros.org/wiki/xacro">
-  <xacro:macro name="yaskawa_common_ros2_control_macro" params="
+  <xacro:macro name="motoman_common_ros2_control_macro" params="
                name
                prefix

File: motoman_ros2_control_support/urdf/common_motoman.xacro (robot description, xacro)
@@ -15,6 +15,6 @@
   <!-- convert to property to use substitution in function -->
   <xacro:include filename="$(find ${description_package})/urdf/${description_macro_file}"/>
-  <xacro:include filename="$(find yaskawa_ros2_control_support)/urdf/common_macro.ros2_control.xacro"/>
-  <xacro:yaskawa_common_ros2_control_macro
+  <xacro:include filename="$(find motoman_ros2_control_support)/urdf/common_macro.ros2_control.xacro"/>
+  <xacro:motoman_common_ros2_control_macro
     name="$(arg robot_name)"
     prefix="$(arg prefix)"

Commit message: Modify the ros2_control support

File: motoman_ros2_control_support/urdf/common_macro.ros2_control.xacro (robot description, xacro)
@@ -4,9 +4,6 @@
                name
                prefix
-               use_mock_hardware:=^|false
-               sim_gazebo_classic:=^|false
-               sim_gazebo:=^|false
-               simulation_controllers
-               description_package"
+               use_mock_hardware:=^|true
+               "
                >
     <ros2_control name="${name}" type="system">
@@ -15,12 +12,6 @@
           <plugin>mock_components/GenericSystem</plugin>
         </xacro:if>
-        <xacro:if value="${sim_gazebo_classic}">
-          <plugin>gazebo_ros2_control/GazeboSystem</plugin>
-        </xacro:if>
-        <xacro:if value="${sim_gazebo}">
-          <plugin>ign_ros2_control/IgnitionSystem</plugin>
-        </xacro:if>
       </hardware>
-    <joint name="${prefix}joint_1">
+    <joint name="${prefix}joint_s">
         <command_interface name="position">
           <param name="min">-1</param>
@@ -31,5 +22,5 @@
         </state_interface>
       </joint>
-      <joint name="${prefix}joint_2">
+      <joint name="${prefix}joint_l">
         <command_interface name="position">
           <param name="min">-1</param>
@@ -40,5 +31,5 @@
         </state_interface>
 	  </joint>
-      <joint name="${prefix}joint_3">
+      <joint name="${prefix}joint_u">
         <command_interface name="position">
           <param name="min">-1</param>
@@ -49,5 +40,5 @@
         </state_interface>
 	  </joint>
-      <joint name="${prefix}joint_4">
+      <joint name="${prefix}joint_r">
         <command_interface name="position">
           <param name="min">-1</param>
@@ -58,5 +49,5 @@
         </state_interface>
       </joint>
-      <joint name="${prefix}joint_5">
+      <joint name="${prefix}joint_b">
         <command_interface name="position">
           <param name="min">-1</param>
@@ -67,5 +58,5 @@
         </state_interface>
       </joint>
-      <joint name="${prefix}joint_6">
+      <joint name="${prefix}joint_t">
         <command_interface name="position">
           <param name="min">-1</param>
@@ -77,25 +68,4 @@
       </joint>
     </ros2_control>
-    <xacro:if value="$(arg sim_gazebo_classic)">
-      <!-- Gazebo plugins -->
-      <gazebo reference="world">
-      </gazebo>
-      <gazebo>
-        <plugin filename="libgazebo_ros2_control.so" name="gazebo_ros2_control">
-          <parameters>${simulation_controllers}</parameters>
-        </plugin>
-      </gazebo>
-    </xacro:if>
-    <xacro:if value="$(arg sim_gazebo)">
-      <!-- Gazebo plugins -->
-      <gazebo reference="world">
-      </gazebo>
-      <gazebo>
-        <plugin filename="libign_ros2_control-system.so" name="ign_ros2_control::IgnitionROS2ControlPlugin">
-          <parameters>${simulation_controllers}</parameters>
-          <controller_manager_node_name>${prefix}controller_manager</controller_manager_node_name>
-        </plugin>
-      </gazebo>
-    </xacro:if>
   </xacro:macro>
 </robot>

Commit message: bkp joints with suffixes

File: motoman_ros2_control_support/urdf/common_macro.ros2_control.xacro (robot description, xacro)
@@ -4,4 +4,5 @@
                name
                prefix
+               joints_with_suffix:=^|false
                use_mock_hardware:=^|false
                sim_gazebo_classic:=^|false
@@ -10,4 +11,18 @@
                description_package"
                >
+    <xacro:property name="joint_1_suffix" value=""/>
+    <xacro:property name="joint_2_suffix" value=""/>
+    <xacro:property name="joint_3_suffix" value=""/>
+    <xacro:property name="joint_4_suffix" value=""/>
+    <xacro:property name="joint_5_suffix" value=""/>
+    <xacro:property name="joint_6_suffix" value=""/>
+    <xacro:if value="${joints_with_suffix}">
+      <xacro:property name="joint_1_suffix" value="_s"/>
+      <xacro:property name="joint_2_suffix" value="_l"/>
+      <xacro:property name="joint_3_suffix" value="_u"/>
+      <xacro:property name="joint_4_suffix" value="_r"/>
+      <xacro:property name="joint_5_suffix" value="_b"/>
+      <xacro:property name="joint_6_suffix" value="_t"/>
+    </xacro:if>
     <ros2_control name="${name}" type="system">
       <hardware>
@@ -22,5 +37,5 @@
         </xacro:if>
       </hardware>
-    <joint name="${prefix}joint_1">
+    <joint name="${prefix}joint_1${joint_1_suffix}">
         <command_interface name="position">
         </command_interface>
@@ -29,5 +44,5 @@
         </state_interface>
       </joint>
-      <joint name="${prefix}joint_2">
+      <joint name="${prefix}joint_2${joint_2_suffix}">
         <command_interface name="position">
         </command_interface>
@@ -36,5 +51,5 @@
         </state_interface>
 	  </joint>
-      <joint name="${prefix}joint_3">
+      <joint name="${prefix}joint_3${joint_3_suffix}">
         <command_interface name="position">
         </command_interface>
@@ -43,5 +58,5 @@
         </state_interface>
 	  </joint>
-      <joint name="${prefix}joint_4">
+      <joint name="${prefix}joint_4${joint_4_suffix}">
         <command_interface name="position">
         </command_interface>
@@ -50,5 +65,5 @@
         </state_interface>
       </joint>
-      <joint name="${prefix}joint_5">
+      <joint name="${prefix}joint_5${joint_5_suffix}">
         <command_interface name="position">
         </command_interface>
@@ -57,5 +72,5 @@
         </state_interface>
       </joint>
-      <joint name="${prefix}joint_6">
+      <joint name="${prefix}joint_6${joint_6_suffix}">
         <command_interface name="position">
         </command_interface>

File: motoman_ros2_control_support/urdf/common_motoman.xacro (robot description, xacro)
@@ -3,4 +3,5 @@
   <xacro:arg name="robot_name" default="yaskawa" />
   <xacro:arg name="prefix" default="" />
+  <xacro:arg name="joints_with_suffix" default="false" />
   <xacro:arg name="description_package" default="" />
   <xacro:arg name="description_macro_file" default="" />
@@ -19,4 +20,5 @@
     name="$(arg robot_name)"
     prefix="$(arg prefix)"
+    joints_with_suffix="$(arg joints_with_suffix)"
     use_mock_hardware="$(arg use_mock_hardware)"
     sim_gazebo_classic="$(arg sim_gazebo_classic)"

Commit message: temporary disable ros2_control when use_mock_hardware or sim_gazebo is used

File: motoman_ros2_control_support/urdf/common_macro.ros2_control.xacro (robot description, xacro)
@@ -25,88 +25,88 @@
       <xacro:property name="joint_6_suffix" value="_t"/>
     </xacro:if>
-    <ros2_control name="${name}" type="system">
-      <hardware>
-        <xacro:if value="${sim_gazebo}">
-          <plugin>gz_ros2_control/GazeboSimSystem</plugin>
-        </xacro:if>
-        <xacro:unless value="${sim_gazebo}">
+    <xacro:if value="${use_mock_hardware or sim_gazebo}">
+      <ros2_control name="${name}" type="system">
+        <hardware>
+          <xacro:if value="${sim_gazebo}">
+            <plugin>gz_ros2_control/GazeboSimSystem</plugin>
+          </xacro:if>
           <xacro:if value="${use_mock_hardware}">
             <plugin>mock_components/GenericSystem</plugin>
           </xacro:if>
-          <xacro:if value="${sim_gazebo_classic}">
-            <plugin>gazebo_ros2_control/GazeboSystem</plugin>
-          </xacro:if>
-        </xacro:unless>
-      </hardware>
-    <joint name="${prefix}joint_1${joint_1_suffix}">
-        <command_interface name="position"/>
-        <state_interface name="position">
-          <param name="initial_value">0</param>
-        </state_interface>
-        <command_interface name="velocity"/>
-        <state_interface name="velocity"/>
+          <xacro:unless value="${use_mock_hardware or sim_gazebo}">
+            <plugin>motoman_hardware_inteface/MotoROS2HardwareInterface</plugin>
+          </xacro:unless>
+        </hardware>
+      <joint name="${prefix}joint_1${joint_1_suffix}">
+          <command_interface name="position"/>
+          <state_interface name="position">
+            <param name="initial_value">0</param>
+          </state_interface>
+          <command_interface name="velocity"/>
+          <state_interface name="velocity"/>
+        </joint>
+        <joint name="${prefix}joint_2${joint_2_suffix}">
+          <command_interface name="position"/>
+          <state_interface name="position">
+            <param name="initial_value">0</param>
+          </state_interface>
+          <command_interface name="velocity"/>
+          <state_interface name="velocity"/>
       </joint>
-      <joint name="${prefix}joint_2${joint_2_suffix}">
-        <command_interface name="position"/>
-        <state_interface name="position">
-          <param name="initial_value">0</param>
-        </state_interface>
-        <command_interface name="velocity"/>
-        <state_interface name="velocity"/>
-	  </joint>
-      <joint name="${prefix}joint_3${joint_3_suffix}">
-        <command_interface name="position"/>
-        <state_interface name="position">
-          <param name="initial_value">0</param>
-        </state_interface>
-        <command_interface name="velocity"/>
-        <state_interface name="velocity"/>
-	  </joint>
-      <joint name="${prefix}joint_4${joint_4_suffix}">
-        <command_interface name="position"/>
-        <state_interface name="position">
-          <param name="initial_value">0</param>
-        </state_interface>
-        <command_interface name="velocity"/>
-        <state_interface name="velocity"/>
+        <joint name="${prefix}joint_3${joint_3_suffix}">
+          <command_interface name="position"/>
+          <state_interface name="position">
+            <param name="initial_value">0</param>
+          </state_interface>
+          <command_interface name="velocity"/>
+          <state_interface name="velocity"/>
       </joint>
-      <joint name="${prefix}joint_5${joint_5_suffix}">
-        <command_interface name="position"/>
-        <state_interface name="position">
-          <param name="initial_value">0</param>
-        </state_interface>
-        <command_interface name="velocity"/>
-        <state_interface name="velocity"/>
-      </joint>
-      <joint name="${prefix}joint_6${joint_6_suffix}">
-        <command_interface name="position"/>
-        <state_interface name="position">
-          <param name="initial_value">0</param>
-        </state_interface>
-        <command_interface name="velocity"/>
-        <state_interface name="velocity"/>
-      </joint>
-      <sensor name="force_torque_sensor">            <!-- Remove/change sensors as needed -->
-        <state_interface name="force.x"/>
-        <state_interface name="force.y"/>
-        <state_interface name="force.z"/>
-        <state_interface name="torque.x"/>
-        <state_interface name="torque.y"/>
-        <state_interface name="torque.z"/>
-        <param name="frame_id">tool0</param>    <!-- Change sensors as needed -->
-        <param name="min_fx">-100</param>
-        <param name="max_fx">100</param>
-        <param name="min_fy">-100</param>
-        <param name="max_fy">100</param>
-        <param name="min_fz">-200</param>
-        <param name="max_fz">200</param>
-        <param name="min_tx">-10</param>
-        <param name="max_tx">10</param>
-        <param name="min_ty">-10</param>
-        <param name="max_ty">10</param>
-        <param name="min_tz">-15</param>
-        <param name="max_tz">15</param>
-      </sensor>
-    </ros2_control>
+        <joint name="${prefix}joint_4${joint_4_suffix}">
+          <command_interface name="position"/>
+          <state_interface name="position">
+            <param name="initial_value">0</param>
+          </state_interface>
+          <command_interface name="velocity"/>
+          <state_interface name="velocity"/>
+        </joint>
+        <joint name="${prefix}joint_5${joint_5_suffix}">
+          <command_interface name="position"/>
+          <state_interface name="position">
+            <param name="initial_value">0</param>
+          </state_interface>
+          <command_interface name="velocity"/>
+          <state_interface name="velocity"/>
+        </joint>
+        <joint name="${prefix}joint_6${joint_6_suffix}">
+          <command_interface name="position"/>
+          <state_interface name="position">
+            <param name="initial_value">0</param>
+          </state_interface>
+          <command_interface name="velocity"/>
+          <state_interface name="velocity"/>
+        </joint>
+        <sensor name="force_torque_sensor">            <!-- Remove/change sensors as needed -->
+          <state_interface name="force.x"/>
+          <state_interface name="force.y"/>
+          <state_interface name="force.z"/>
+          <state_interface name="torque.x"/>
+          <state_interface name="torque.y"/>
+          <state_interface name="torque.z"/>
+          <param name="frame_id">tool0</param>    <!-- Change sensors as needed -->
+          <param name="min_fx">-100</param>
+          <param name="max_fx">100</param>
+          <param name="min_fy">-100</param>
+          <param name="max_fy">100</param>
+          <param name="min_fz">-200</param>
+          <param name="max_fz">200</param>
+          <param name="min_tx">-10</param>
+          <param name="max_tx">10</param>
+          <param name="min_ty">-10</param>
+          <param name="max_ty">10</param>
+          <param name="min_tz">-15</param>
+          <param name="max_tz">15</param>
+        </sensor>
+      </ros2_control>
+    </xacro:if>
     <xacro:if value="$(arg sim_gazebo_classic)">
       <!-- Gazebo plugins -->

Commit message: adjust ros2_control macro to start MotoROS2HardwareInterface

File: motoman_ros2_control_support/urdf/common_macro.ros2_control.xacro (robot description, xacro)
@@ -25,6 +25,6 @@
       <xacro:property name="joint_6_suffix" value="_t"/>
     </xacro:if>
-    <xacro:if value="${use_mock_hardware or sim_gazebo}">
-      <ros2_control name="${name}" type="system">
+    <!-- <xacro:if value="${use_mock_hardware or sim_gazebo}"> -->
+      <ros2_control name="${name}" type="system" is_async="true">
         <hardware>
           <xacro:if value="${sim_gazebo}">
@@ -35,8 +35,11 @@
           </xacro:if>
           <xacro:unless value="${use_mock_hardware or sim_gazebo}">
-            <plugin>motoman_hardware_inteface/MotoROS2HardwareInterface</plugin>
+            <!-- <plugin>motoman_hardware_inteface/MotoROS2HardwareInterface</plugin> -->
+            <plugin>iaa_hardware_interfaces/MotoROS2HardwareInterface</plugin>
+            <param name="queue_traj_point_srv_name">/queue_traj_point</param>
+            <param name="joint_states_topic_name">/hc20sdtp/joint_states</param>
           </xacro:unless>
         </hardware>
-      <joint name="${prefix}joint_1${joint_1_suffix}">
+        <joint name="${prefix}joint_1${joint_1_suffix}">
           <command_interface name="position"/>
           <state_interface name="position">
@@ -53,5 +56,5 @@
           <command_interface name="velocity"/>
           <state_interface name="velocity"/>
-      </joint>
+        </joint>
         <joint name="${prefix}joint_3${joint_3_suffix}">
           <command_interface name="position"/>
@@ -61,5 +64,5 @@
           <command_interface name="velocity"/>
           <state_interface name="velocity"/>
-      </joint>
+        </joint>
         <joint name="${prefix}joint_4${joint_4_suffix}">
           <command_interface name="position"/>
@@ -86,27 +89,29 @@
           <state_interface name="velocity"/>
         </joint>
-        <sensor name="force_torque_sensor">            <!-- Remove/change sensors as needed -->
-          <state_interface name="force.x"/>
-          <state_interface name="force.y"/>
-          <state_interface name="force.z"/>
-          <state_interface name="torque.x"/>
-          <state_interface name="torque.y"/>
-          <state_interface name="torque.z"/>
-          <param name="frame_id">tool0</param>    <!-- Change sensors as needed -->
-          <param name="min_fx">-100</param>
-          <param name="max_fx">100</param>
-          <param name="min_fy">-100</param>
-          <param name="max_fy">100</param>
-          <param name="min_fz">-200</param>
-          <param name="max_fz">200</param>
-          <param name="min_tx">-10</param>
-          <param name="max_tx">10</param>
-          <param name="min_ty">-10</param>
-          <param name="max_ty">10</param>
-          <param name="min_tz">-15</param>
-          <param name="max_tz">15</param>
-        </sensor>
+        <xacro:if value="${use_mock_hardware or sim_gazebo}">
+          <sensor name="force_torque_sensor">
+            <state_interface name="force.x"/>
+            <state_interface name="force.y"/>
+            <state_interface name="force.z"/>
+            <state_interface name="torque.x"/>
+            <state_interface name="torque.y"/>
+            <state_interface name="torque.z"/>
+            <param name="frame_id">tool0</param>
+            <param name="min_fx">-100</param>
+            <param name="max_fx">100</param>
+            <param name="min_fy">-100</param>
+            <param name="max_fy">100</param>
+            <param name="min_fz">-200</param>
+            <param name="max_fz">200</param>
+            <param name="min_tx">-10</param>
+            <param name="max_tx">10</param>
+            <param name="min_ty">-10</param>
+            <param name="max_ty">10</param>
+            <param name="min_tz">-15</param>
+            <param name="max_tz">15</param>
+          </sensor>
+        </xacro:if>
       </ros2_control>
-    </xacro:if>
+    <!-- </xacro:if> -->
     <xacro:if value="$(arg sim_gazebo_classic)">
       <!-- Gazebo plugins -->

Commit message: update fts ros2_control macro

File: motoman_ros2_control_support/urdf/common_macro.ros2_control.xacro (robot description, xacro)
@@ -24,4 +24,27 @@
       <xacro:property name="joint_6_suffix" value="_t"/>
     </xacro:if>
+    <xacro:property name="sensor_block">
+      <sensor name="force_torque_sensor">
+        <state_interface name="force.x"/>
+        <state_interface name="force.y"/>
+        <state_interface name="force.z"/>
+        <state_interface name="torque.x"/>
+        <state_interface name="torque.y"/>
+        <state_interface name="torque.z"/>
+        <param name="frame_id">tool0</param>
+        <param name="min_fx">-100</param>
+        <param name="max_fx">100</param>
+        <param name="min_fy">-100</param>
+        <param name="max_fy">100</param>
+        <param name="min_fz">-200</param>
+        <param name="max_fz">200</param>
+        <param name="min_tx">-10</param>
+        <param name="max_tx">10</param>
+        <param name="min_ty">-10</param>
+        <param name="max_ty">10</param>
+        <param name="min_tz">-15</param>
+        <param name="max_tz">15</param>
+      </sensor>
+    </xacro:property>
       <ros2_control name="${name}" type="system" is_async="${not (use_mock_hardware or sim_gazebo)}" >
       <!-- <ros2_control name="${name}" type="system" is_async="false" > -->
@@ -89,28 +112,23 @@
         </joint>
         <xacro:if value="${use_mock_hardware or sim_gazebo}">
-          <sensor name="force_torque_sensor">
-            <state_interface name="force.x"/>
-            <state_interface name="force.y"/>
-            <state_interface name="force.z"/>
-            <state_interface name="torque.x"/>
-            <state_interface name="torque.y"/>
-            <state_interface name="torque.z"/>
-            <param name="frame_id">tool0</param>
-            <param name="min_fx">-100</param>
-            <param name="max_fx">100</param>
-            <param name="min_fy">-100</param>
-            <param name="max_fy">100</param>
-            <param name="min_fz">-200</param>
-            <param name="max_fz">200</param>
-            <param name="min_tx">-10</param>
-            <param name="max_tx">10</param>
-            <param name="min_ty">-10</param>
-            <param name="max_ty">10</param>
-            <param name="min_tz">-15</param>
-            <param name="max_tz">15</param>
-          </sensor>
+          <xacro:insert_block name="sensor_block"/>
         </xacro:if>
       </ros2_control>
     <!-- </xacro:if> -->
+    <xacro:if value="${not (use_mock_hardware or sim_gazebo)}" >
+      <ros2_control name="fts_hw" type="sensor" is_async="true" >
+        <hardware>
+          <plugin>iaa_hardware_interfaces/FTSHardwareInterface</plugin>
+          <param name="fts_topic">/tcp_force_torque</param>
+          <param name="force_x_name">force.x</param>
+          <param name="force_y_name">force.y</param>
+          <param name="force_z_name">force.z</param>
+          <param name="torque_x_name">torque.x</param>
+          <param name="torque_y_name">torque.y</param>
+          <param name="torque_z_name">torque.z</param>
+        </hardware>
+        <xacro:insert_block name="sensor_block"/>
+      </ros2_control>
+    </xacro:if>
     <xacro:if value="$(arg sim_gazebo)">
       <!-- Gazebo plugins -->
