Commit message: clean tabs

File: motoman_ros2_control_support/urdf/common_macro.ros2_control.xacro (robot description, xacro)
@@ -47,73 +47,72 @@
       </sensor>
     </xacro:property>
-      <ros2_control name="${name}" type="system" is_async="${not (use_mock_hardware or sim_gazebo)}" >
-      <!-- <ros2_control name="${name}" type="system" is_async="false" > -->
-        <hardware>
-          <xacro:if value="${sim_gazebo}">
-            <plugin>gz_ros2_control/GazeboSimSystem</plugin>
-          </xacro:if>
-          <xacro:if value="${use_mock_hardware}">
-            <plugin>mock_components/GenericSystem</plugin>
-          </xacro:if>
-          <xacro:unless value="${use_mock_hardware or sim_gazebo}">
-            <!-- <plugin>motoman_hardware_inteface/MotoROS2HardwareInterface</plugin> -->
-            <plugin>iaa_hardware_interfaces/MotoROS2HardwareInterface</plugin>
-            <param name="queue_traj_point_srv_name">/queue_traj_point</param>
-            <param name="joint_states_topic_name">/hc20sdtp_joint_states</param>
-          </xacro:unless>
-        </hardware>
-        <joint name="${prefix}joint_1${joint_1_suffix}">
-          <command_interface name="position"/>
-          <state_interface name="position">
-            <param name="initial_value">0</param>
-          </state_interface>
-          <command_interface name="velocity"/>
-          <state_interface name="velocity"/>
-        </joint>
-        <joint name="${prefix}joint_2${joint_2_suffix}">
-          <command_interface name="position"/>
-          <state_interface name="position">
-            <param name="initial_value">0</param>
-          </state_interface>
-          <command_interface name="velocity"/>
-          <state_interface name="velocity"/>
-        </joint>
-        <joint name="${prefix}joint_3${joint_3_suffix}">
-          <command_interface name="position"/>
-          <state_interface name="position">
-            <param name="initial_value">0</param>
-          </state_interface>
-          <command_interface name="velocity"/>
-          <state_interface name="velocity"/>
-        </joint>
-        <joint name="${prefix}joint_4${joint_4_suffix}">
-          <command_interface name="position"/>
-          <state_interface name="position">
-            <param name="initial_value">0</param>
-          </state_interface>
-          <command_interface name="velocity"/>
-          <state_interface name="velocity"/>
-        </joint>
-        <joint name="${prefix}joint_5${joint_5_suffix}">
-          <command_interface name="position"/>
-          <state_interface name="position">
-            <param name="initial_value">0</param>
-          </state_interface>
-          <command_interface name="velocity"/>
-          <state_interface name="velocity"/>
-        </joint>
-        <joint name="${prefix}joint_6${joint_6_suffix}">
-          <command_interface name="position"/>
-          <state_interface name="position">
-            <param name="initial_value">0</param>
-          </state_interface>
-          <command_interface name="velocity"/>
-          <state_interface name="velocity"/>
-        </joint>
-        <xacro:if value="${use_mock_hardware or sim_gazebo}">
-          <xacro:insert_block name="sensor_block"/>
+    <ros2_control name="${name}" type="system" is_async="${not (use_mock_hardware or sim_gazebo)}" >
+    <!-- <ros2_control name="${name}" type="system" is_async="false" > -->
+      <hardware>
+        <xacro:if value="${sim_gazebo}">
+          <plugin>gz_ros2_control/GazeboSimSystem</plugin>
         </xacro:if>
-      </ros2_control>
-    <!-- </xacro:if> -->
+        <xacro:if value="${use_mock_hardware}">
+          <plugin>mock_components/GenericSystem</plugin>
+        </xacro:if>
+        <xacro:unless value="${use_mock_hardware or sim_gazebo}">
+          <!-- <plugin>motoman_hardware_inteface/MotoROS2HardwareInterface</plugin> -->
+          <plugin>iaa_hardware_interfaces/MotoROS2HardwareInterface</plugin>
+          <param name="queue_traj_point_srv_name">/queue_traj_point</param>
+          <param name="joint_states_topic_name">/hc20sdtp_joint_states</param>
+        </xacro:unless>
+      </hardware>
+      <joint name="${prefix}joint_1${joint_1_suffix}">
+        <command_interface name="position"/>
+        <state_interface name="position">
+          <param name="initial_value">0</param>
+        </state_interface>
+        <command_interface name="velocity"/>
+        <state_interface name="velocity"/>
+      </joint>
+      <joint name="${prefix}joint_2${joint_2_suffix}">
+        <command_interface name="position"/>
+        <state_interface name="position">
+          <param name="initial_value">0</param>
+        </state_interface>
+        <command_interface name="velocity"/>
+        <state_interface name="velocity"/>
+      </joint>
+      <joint name="${prefix}joint_3${joint_3_suffix}">
+        <command_interface name="position"/>
+        <state_interface name="position">
+          <param name="initial_value">0</param>
+        </state_interface>
+        <command_interface name="velocity"/>
+        <state_interface name="velocity"/>
+      </joint>
+      <joint name="${prefix}joint_4${joint_4_suffix}">
+        <command_interface name="position"/>
+        <state_interface name="position">
+          <param name="initial_value">0</param>
+        </state_interface>
+        <command_interface name="velocity"/>
+        <state_interface name="velocity"/>
+      </joint>
+      <joint name="${prefix}joint_5${joint_5_suffix}">
+        <command_interface name="position"/>
+        <state_interface name="position">
+          <param name="initial_value">0</param>
+        </state_interface>
+        <command_interface name="velocity"/>
+        <state_interface name="velocity"/>
+      </joint>
+      <joint name="${prefix}joint_6${joint_6_suffix}">
+        <command_interface name="position"/>
+        <state_interface name="position">
+          <param name="initial_value">0</param>
+        </state_interface>
+        <command_interface name="velocity"/>
+        <state_interface name="velocity"/>
+      </joint>
+      <xacro:if value="${use_mock_hardware or sim_gazebo}">
+        <xacro:insert_block name="sensor_block"/>
+      </xacro:if>
+    </ros2_control>
     <xacro:if value="${not (use_mock_hardware or sim_gazebo)}" >
       <ros2_control name="fts_hw" type="sensor" is_async="true" >
@@ -139,11 +138,11 @@
           <parameters>${simulation_controllers}</parameters>
           <controller_manager_node_name>${prefix}controller_manager</controller_manager_node_name>
-            <ros>
-              <!-- <remapping>/position_trajectory_controller/follow_joint_trajectory/_action/feedback:=/follow_joint_trajectory/_action/feedback</remapping>
-              <remapping>/position_trajectory_controller/follow_joint_trajectory/_action/status:=/follow_joint_trajectory/_action/status</remapping>
-              <remapping>/position_trajectory_controller/follow_joint_trajectory/_action/cancel_goal:=/follow_joint_trajectory/_action/cancel_goal</remapping>
-              <remapping>/position_trajectory_controller/follow_joint_trajectory/_action/get_result:=/follow_joint_trajectory/_action/get_result</remapping>
-              <remapping>/position_trajectory_controller/follow_joint_trajectory/_action/send_goal:=/follow_joint_trajectory/_action/send_goal</remapping> -->
-          </ros>
+          <!-- <ros>
+            <remapping>/position_trajectory_controller/follow_joint_trajectory/_action/feedback:=/follow_joint_trajectory/_action/feedback</remapping>
+            <remapping>/position_trajectory_controller/follow_joint_trajectory/_action/status:=/follow_joint_trajectory/_action/status</remapping>
+            <remapping>/position_trajectory_controller/follow_joint_trajectory/_action/cancel_goal:=/follow_joint_trajectory/_action/cancel_goal</remapping>
+            <remapping>/position_trajectory_controller/follow_joint_trajectory/_action/get_result:=/follow_joint_trajectory/_action/get_result</remapping>
+            <remapping>/position_trajectory_controller/follow_joint_trajectory/_action/send_goal:=/follow_joint_trajectory/_action/send_goal</remapping>
+          </ros> -->
         </plugin>
       </gazebo>

Commit message: add passing of initial joint positions when using mock_hw

File: motoman_ros2_control_support/urdf/common_macro.ros2_control.xacro (robot description, xacro)
@@ -9,5 +9,6 @@
                sim_gazebo:=^|false
                simulation_controllers
-               description_package"
+               description_package
+               initial_positions:=${dict(joint_a1=0.0,joint_a2=0.0,joint_a3=0.0,joint_a4=0.0,joint_a5=0.0,joint_a6=0.0)}"
                >
     <xacro:property name="joint_1_suffix" value=""/>
@@ -67,5 +68,5 @@
         <command_interface name="position"/>
         <state_interface name="position">
-          <param name="initial_value">0</param>
+          <param name="initial_value">${initial_positions['joint_a1']}</param>
         </state_interface>
         <command_interface name="velocity"/>
@@ -75,5 +76,5 @@
         <command_interface name="position"/>
         <state_interface name="position">
-          <param name="initial_value">0</param>
+          <param name="initial_value">${initial_positions['joint_a2']}</param>
         </state_interface>
         <command_interface name="velocity"/>
@@ -83,5 +84,5 @@
         <command_interface name="position"/>
         <state_interface name="position">
-          <param name="initial_value">0</param>
+          <param name="initial_value">${initial_positions['joint_a3']}</param>
         </state_interface>
         <command_interface name="velocity"/>
@@ -91,5 +92,5 @@
         <command_interface name="position"/>
         <state_interface name="position">
-          <param name="initial_value">0</param>
+          <param name="initial_value">${initial_positions['joint_a4']}</param>
         </state_interface>
         <command_interface name="velocity"/>
@@ -99,5 +100,5 @@
         <command_interface name="position"/>
         <state_interface name="position">
-          <param name="initial_value">0</param>
+          <param name="initial_value">${initial_positions['joint_a5']}</param>
         </state_interface>
         <command_interface name="velocity"/>
@@ -107,5 +108,5 @@
         <command_interface name="position"/>
         <state_interface name="position">
-          <param name="initial_value">0</param>
+          <param name="initial_value">${initial_positions['joint_a6']}</param>
         </state_interface>
         <command_interface name="velocity"/>

File: motoman_ros2_control_support/urdf/common_motoman.xacro (robot description, xacro)
@@ -16,4 +16,5 @@
   <!-- convert to property to use substitution in function -->
   <xacro:include filename="$(find ${description_package})/urdf/${description_macro_file}"/>
+  <xacro:property name="initial_positions_file" value="$(find ${description_package})/config/initial_positions.yaml"/>
   <xacro:include filename="$(find motoman_ros2_control_support)/urdf/common_macro.ros2_control.xacro"/>
   <xacro:if value="$(arg use_mock_hardware)">
@@ -27,4 +28,5 @@
       simulation_controllers="$(arg simulation_controllers)"
       description_package="$(arg description_package)"
+      initial_positions="${xacro.load_yaml(initial_positions_file)}"
     />
   </xacro:if>
